File: pcbfiles/pcb.kicad_pcb (KiCad board)
At the start: 2 copper layers, 0 parts

Commit message: continue schematic, test pcb idea
Parts:
- added REF**: PinHeader_1x12_P2.54mm_Vertical, Connector_PinHeader_2.54mm:PinHeader_1x12_P2.54mm_Vertical, F.Cu at (237.2, -68.1)
- added REF**: 1U, MX_Only:MXOnly-1U-Hotswap, F.Cu at (242.9, -118.3)
- added REF**: PinHeader_1x12_P2.54mm_Vertical, Connector_PinHeader_2.54mm:PinHeader_1x12_P2.54mm_Vertical, F.Cu at (189.5, -69.7)
- added REF**: 1.25U, MX_Only:MXOnly-1.25U-Hotswap, F.Cu at (258.6, -53.0)
- added REF**: 1.25U, MX_Only:MXOnly-1.25U-Hotswap, F.Cu at (218.1, -54.6)
- added REF**: 1.25U, MX_Only:MXOnly-1.25U-Hotswap, F.Cu at (239.6, -53.0)
- added REF**: 2.25U, MX_Only:MXOnly-2.25U-Hotswap-ReversedStabilizers, F.Cu at (211.9, -117.5)
- added REF**: PinHeader_1x12_P2.54mm_Vertical, Connector_PinHeader_2.54mm:PinHeader_1x12_P2.54mm_Vertical, F.Cu at (240.5, -111.9)
- added REF**: PinHeader_1x12_P2.54mm_Vertical, Connector_PinHeader_2.54mm:PinHeader_1x12_P2.54mm_Vertical, F.Cu at (192.9, -113.5)
- added REF**: 1.5U, MX_Only:MXOnly-1.5U-Hotswap, F.Cu at (261.9, -123.0)

Commit message: PCB Layout, Diodes, Matrix
Main body switches placed, some parts of matrix routed, PCB progress.
Parts:
- removed the REF** at (237.2, -68.1)
- removed the REF** at (242.9, -118.3)
- removed the REF** at (189.5, -69.7)
- removed the REF** at (258.6, -53.0)
- removed the REF** at (218.1, -54.6)
- removed the REF** at (239.6, -53.0)
- removed the REF** at (211.9, -117.5)
- removed the REF** at (240.5, -111.9)
- removed the REF** at (192.9, -113.5)
- removed the REF** at (261.9, -123.0)
- added C1: 4.7uF, Capacitor_SMD:C_0805_2012Metric, F.Cu at (289.3, 227.8)
- added C2: 4.7n, Capacitor_SMD:C_0805_2012Metric, B.Cu at (491.3, -71.5)
- added C3: 1uF, Capacitor_SMD:C_0805_2012Metric, B.Cu at (528.8, -34.5)
- added C4: 1uF, Capacitor_SMD:C_0805_2012Metric, B.Cu at (445.1, -118.6)
- added C5: 4.7n, Capacitor_SMD:C_0805_2012Metric, B.Cu at (465.4, -98.4)
- added C6: 4.7uF, Capacitor_SMD:C_0805_2012Metric, B.Cu at (485.6, -78.2)
- added C7: 1uF, Capacitor_SMD:C_0805_2012Metric, B.Cu at (543.2, -20.9)
- added C8: 1uF, Capacitor_SMD:C_0805_2012Metric, B.Cu at (523.0, -41.2)
- added D1: 1N5819, Diode_SMD:D_SOD-123, B.Cu at (500.6, -38.6)
- added D10: D_Small, Diode_SMD:D_SOD-123, B.Cu at (22.2, 0.00)
- added D11: D_Small, Diode_SMD:D_SOD-123, B.Cu at (22.2, 19.1)
- added D12: D_Small, Diode_SMD:D_SOD-123, B.Cu at (22.2, 38.1)
- added D13: D_Small, Diode_SMD:D_SOD-123, B.Cu at (22.2, 57.1)
- added D14: D_Small, Diode_SMD:D_SOD-123, B.Cu at (22.2, 76.2)
- added D15: D_Small, Diode_SMD:D_SOD-123, B.Cu at (534.3, -24.7)
- added D16: D_Small, Diode_SMD:D_SOD-123, B.Cu at (41.3, -2.38)
- added D17: D_Small, Diode_SMD:D_SOD-123, B.Cu at (41.3, 16.7)
- added D18: D_Small, Diode_SMD:D_SOD-123, B.Cu at (41.3, 35.7)
- added D19: D_Small, Diode_SMD:D_SOD-123, B.Cu at (41.3, 54.8)
- added D2: D_Small, Diode_SMD:D_SOD-123, B.Cu at (561.2, 19.3)
- added D20: D_Small, Diode_SMD:D_SOD-123, B.Cu at (41.3, 73.8)
- added D21: D_Small, Diode_SMD:D_SOD-123, B.Cu at (60.3, -4.76)
- added D22: D_Small, Diode_SMD:D_SOD-123, B.Cu at (60.3, 14.3)
- added D23: D_Small, Diode_SMD:D_SOD-123, B.Cu at (60.3, 33.3)
- added D24: D_Small, Diode_SMD:D_SOD-123, B.Cu at (60.3, 52.4)
- added D25: D_Small, Diode_SMD:D_SOD-123, B.Cu at (60.3, 71.4)
- added D26: D_Small, Diode_SMD:D_SOD-123, B.Cu at (67.5, 92.9)
- added D27: D_Small, Diode_SMD:D_SOD-123, B.Cu at (79.4, -2.38)
- added D28: D_Small, Diode_SMD:D_SOD-123, B.Cu at (79.4, 16.7)
- added D29: D_Small, Diode_SMD:D_SOD-123, B.Cu at (79.4, 35.7)
- added D3: D_Small, Diode_SMD:D_SOD-123, B.Cu at (3.17, 0.00)
- added D30: D_Small, Diode_SMD:D_SOD-123, B.Cu at (79.4, 54.8)
- added D31: D_Small, Diode_SMD:D_SOD-123, B.Cu at (79.4, 73.8)
- added D32: D_Small, Diode_SMD:D_SOD-123, B.Cu at (206.4, 150.0)
- added D33: D_Small, Diode_SMD:D_SOD-123, B.Cu at (98.4, 0.00)
- added D34: D_Small, Diode_SMD:D_SOD-123, B.Cu at (98.4, 19.1)
- added D35: D_Small, Diode_SMD:D_SOD-123, B.Cu at (98.4, 38.1)
- added D36: D_Small, Diode_SMD:D_SOD-123, B.Cu at (98.4, 57.1)
- added D37: D_Small, Diode_SMD:D_SOD-123, B.Cu at (98.4, 76.2)
- added D38: D_Small, Diode_SMD:D_SOD-123, B.Cu at (98.4, 95.2)
- added D39: LED_Small, Diode_SMD:D_0805_2012Metric, B.Cu at (491.3, -57.9)
- added D4: D_Small, Diode_SMD:D_SOD-123, B.Cu at (3.17, 19.1)
- added D40: SR05, Package_TO_SOT_SMD:SOT-143, B.Cu at (551.8, -11.7)
- added D41: D_Small, Diode_SMD:D_SOD-123, B.Cu at (331.8, 175.4)
- added D42: D_Small, Diode_SMD:D_SOD-123, B.Cu at (117.5, 9.53)
- added D43: D_Small, Diode_SMD:D_SOD-123, B.Cu at (118.3, 42.9)
- added D44: D_Small, Diode_SMD:D_SOD-123, B.Cu at (118.3, 76.2)
- added D45: D_Small, Diode_SMD:D_SOD-123, B.Cu at (118.3, 100.0)
- added D46: D_Small, Diode_SMD:D_SOD-123, B.Cu at (325.4, 173.0)
- added D47: SR05, Package_TO_SOT_SMD:SOT-143, B.Cu at (534.0, -28.6)
- added D48: LED_Small, Diode_SMD:D_0805_2012Metric, B.Cu at (557.2, -7.55)
- added D49: D_Small, Diode_SMD:D_SOD-123, B.Cu at (155.6, 9.53)
- added D5: D_Small, Diode_SMD:D_SOD-123, B.Cu at (3.17, 38.1)
- added D50: D_Small, Diode_SMD:D_SOD-123, B.Cu at (158.0, 36.5)
- added D51: D_Small, Diode_SMD:D_SOD-123, B.Cu at (512.1, -41.3)
- added D52: D_Small, Diode_SMD:D_SOD-123, B.Cu at (500.6, -52.0)
- added D53: D_Small, Diode_SMD:D_SOD-123, B.Cu at (532.4, -21.3)
- added D54: D_Small, Diode_SMD:D_SOD-123, B.Cu at (174.6, 0.00)
- added D55: D_Small, Diode_SMD:D_SOD-123, B.Cu at (174.6, 19.1)
- added D56: D_Small, Diode_SMD:D_SOD-123, B.Cu at (174.6, 38.1)
- added D57: D_Small, Diode_SMD:D_SOD-123, B.Cu at (174.6, 57.1)
- added D58: D_Small, Diode_SMD:D_SOD-123, B.Cu at (174.6, 76.2)
- added D59: D_Small, Diode_SMD:D_SOD-123, B.Cu at (174.6, 95.2)
- added D6: D_Small, Diode_SMD:D_SOD-123, B.Cu at (3.17, 57.1)
- added D60: 1N5819, Diode_SMD:D_SOD-123, B.Cu at (500.6, -48.6)
- added D61: D_Small, Diode_SMD:D_SOD-123, B.Cu at (242.9, 182.6)
- added D62: D_Small, Diode_SMD:D_SOD-123, B.Cu at (480.4, -68.3)
- added D63: D_Small, Diode_SMD:D_SOD-123, B.Cu at (193.7, -2.38)
- added D64: D_Small, Diode_SMD:D_SOD-123, B.Cu at (193.7, 16.7)
- added D65: D_Small, Diode_SMD:D_SOD-123, B.Cu at (193.7, 35.7)
- added D66: D_Small, Diode_SMD:D_SOD-123, B.Cu at (193.7, 54.8)
- added D67: D_Small, Diode_SMD:D_SOD-123, B.Cu at (193.7, 73.8)
- added D68: D_Small, Diode_SMD:D_SOD-123, B.Cu at (561.2, 15.9)
- added D69: D_Small, Diode_SMD:D_SOD-123, B.Cu at (212.7, -4.76)
- added D7: D_Small, Diode_SMD:D_SOD-123, B.Cu at (3.17, 76.2)
- added D70: D_Small, Diode_SMD:D_SOD-123, B.Cu at (212.7, 14.3)
- added D71: D_Small, Diode_SMD:D_SOD-123, B.Cu at (212.7, 33.3)
- added D72: D_Small, Diode_SMD:D_SOD-123, B.Cu at (212.7, 52.4)
- added D73: D_Small, Diode_SMD:D_SOD-123, B.Cu at (212.7, 71.4)
- added D74: D_Small, Diode_SMD:D_SOD-123, B.Cu at (210.3, 92.9)
- added D75: D_Small, Diode_SMD:D_SOD-123, B.Cu at (231.8, -2.38)
- added D76: D_Small, Diode_SMD:D_SOD-123, B.Cu at (231.8, 16.7)
- added D77: D_Small, Diode_SMD:D_SOD-123, B.Cu at (231.8, 35.7)
- added D78: D_Small, Diode_SMD:D_SOD-123, B.Cu at (231.8, 54.8)
- added D79: D_Small, Diode_SMD:D_SOD-123, B.Cu at (231.8, 73.8)
- added D8: D_Small, Diode_SMD:D_SOD-123, B.Cu at (445.8, -115.4)
- added D80: D_Small, Diode_SMD:D_SOD-123, B.Cu at (250.8, 0.00)
- added D81: D_Small, Diode_SMD:D_SOD-123, B.Cu at (250.8, 19.1)
- added D82: D_Small, Diode_SMD:D_SOD-123, B.Cu at (250.8, 38.1)
- added D83: D_Small, Diode_SMD:D_SOD-123, B.Cu at (250.8, 57.1)
- added D84: D_Small, Diode_SMD:D_SOD-123, B.Cu at (250.8, 76.2)
- added D85: D_Small, Diode_SMD:D_SOD-123, B.Cu at (517.9, -41.3)
- added D86: D_Small, Diode_SMD:D_SOD-123, B.Cu at (269.9, 0.00)
- added D87: D_Small, Diode_SMD:D_SOD-123, B.Cu at (259.6, 21.4)
- added D88: D_Small, Diode_SMD:D_SOD-123, B.Cu at (269.9, 38.1)
- added D89: D_Small, Diode_SMD:D_SOD-123, B.Cu at (269.9, 57.1)
- added D9: D_Small, Diode_SMD:D_SOD-123, B.Cu at (523.6, -34.7)
- added D90: D_Small, Diode_SMD:D_SOD-123, B.Cu at (269.9, 76.2)
- added D91: D_Small, Diode_SMD:D_SOD-123, B.Cu at (561.2, 29.3)
- added D92: D_Small, Diode_SMD:D_SOD-123, B.Cu at (561.2, 26.0)
- added F1: 500ma, Fuse:Fuse_1206_3216Metric, B.Cu at (506.3, -55.3)
- added F2: 500ma, Fuse:Fuse_1206_3216Metric, B.Cu at (523.6, -38.0)
- added J1: Conn_01x04_Female, Connector_PinHeader_2.54mm:PinHeader_1x04_P2.54mm_Vertical, F.Cu at (282.6, 214.6)
- added J6: Conn_01x04_Female, Connector_PinHeader_2.54mm:PinHeader_1x04_P2.54mm_Vertical, F.Cu at (277.9, 214.6)
- added Q1: AO3401A, Package_TO_SOT_SMD:SOT-23, B.Cu at (459.6, -102.5)
- added Q2: AO3401A, Package_TO_SOT_SMD:SOT-23, B.Cu at (439.4, -122.7)
- added R1: 5.1k, Resistor_SMD:R_0805_2012Metric, B.Cu at (439.4, -126.5)
- added R10: 5.1k, Resistor_SMD:R_0805_2012Metric, B.Cu at (476.8, -88.3)
- added R11: 5.1k, Resistor_SMD:R_0805_2012Metric, B.Cu at (456.6, -108.5)
- added R12: 10k, Resistor_SMD:R_0805_2012Metric, B.Cu at (539.4, -24.5)
- added R13: 806k, Resistor_SMD:R_0805_2012Metric, B.Cu at (450.9, -111.9)
- added R14: 1k, Resistor_SMD:R_0805_2012Metric, B.Cu at (511.5, -51.2)
- added R15: 2M, Resistor_SMD:R_0805_2012Metric, B.Cu at (471.1, -91.7)
- added R16: 10k, Resistor_SMD:R_0805_2012Metric, B.Cu at (484.2, -81.5)
- added R2: 10k, Resistor_SMD:R_0805_2012Metric, B.Cu at (443.8, -121.9)
- added R3: 10k, Resistor_SMD:R_0805_2012Metric, B.Cu at (464.0, -101.7)
- added R4: 1M, Resistor_SMD:R_0805_2012Metric, B.Cu at (533.6, -32.4)
- added R5: 5.1k, Resistor_SMD:R_0805_2012Metric, B.Cu at (491.3, -74.5)
- added R6: 1M, Resistor_SMD:R_0805_2012Metric, B.Cu at (471.1, -94.6)
- added R7: 806k, Resistor_SMD:R_0805_2012Metric, B.Cu at (511.5, -54.1)
- added R8: 2M, Resistor_SMD:R_0805_2012Metric, B.Cu at (450.9, -114.8)
- added R9: 1k, Resistor_SMD:R_0805_2012Metric, B.Cu at (497.0, -68.1)
- added REF**: 1U, MX_Only:MXOnly-1U, F.Cu at (133.3, 61.9)
- added SW10: SW_SPST, MX_Only:MXOnly-1U-Hotswap, F.Cu at (19.1, 0.00)
- added SW11: SW_SPST, MX_Only:MXOnly-1U-Hotswap, F.Cu at (19.1, 19.1)
- added SW12: SW_SPST, MX_Only:MXOnly-1U-Hotswap, F.Cu at (19.1, 38.1)
- added SW13: SW_SPST, MX_Only:MXOnly-1U-Hotswap, F.Cu at (19.1, 57.1)
- added SW14: SW_SPST, MX_Only:MXOnly-1U-Hotswap, F.Cu at (19.1, 76.2)
- added SW15: SW_SPST, MX_Only:MXOnly-1U-Hotswap, F.Cu at (449.7, 97.9)
- added SW16: SW_SPST, MX_Only:MXOnly-1U-Hotswap, F.Cu at (38.1, -2.38)
- added SW17: SW_SPST, MX_Only:MXOnly-1U-Hotswap, F.Cu at (38.1, 16.7)
- added SW18: SW_SPST, MX_Only:MXOnly-1U-Hotswap, F.Cu at (38.1, 35.7)
- added SW19: SW_SPST, MX_Only:MXOnly-1U-Hotswap, F.Cu at (38.1, 54.8)
- added SW2: SW_SPST, MX_Only:MXOnly-1U-Hotswap, F.Cu at (429.5, 158.5)
- added SW20: SW_SPST, MX_Only:MXOnly-1U-Hotswap, F.Cu at (38.1, 73.8)
- added SW21: SW_SPST, MX_Only:MXOnly-1U-Hotswap, F.Cu at (57.1, -4.76)
- added SW22: SW_SPST, MX_Only:MXOnly-1U-Hotswap, F.Cu at (57.1, 14.3)
- added SW23: SW_SPST, MX_Only:MXOnly-1U-Hotswap, F.Cu at (57.1, 33.3)
- added SW24: SW_SPST, MX_Only:MXOnly-1U-Hotswap, F.Cu at (57.1, 52.4)
- added SW25: SW_SPST, MX_Only:MXOnly-1U-Hotswap, F.Cu at (57.1, 71.4)
- added SW26: SW_SPST, MX_Only:MXOnly-2.25U-Hotswap-ReversedStabilizers, F.Cu at (64.3, 92.9)
- added SW27: SW_SPST, MX_Only:MXOnly-1U-Hotswap, F.Cu at (76.2, -2.38)
- added SW28: SW_SPST, MX_Only:MXOnly-1U-Hotswap, F.Cu at (76.2, 16.7)
- added SW29: SW_SPST, MX_Only:MXOnly-1U-Hotswap, F.Cu at (76.2, 35.7)
- added SW3: SW_SPST, MX_Only:MXOnly-1U-Hotswap, F.Cu at (0.00, 0.00)
- added SW30: SW_SPST, MX_Only:MXOnly-1U-Hotswap, F.Cu at (76.2, 54.8)
- added SW31: SW_SPST, MX_Only:MXOnly-1U-Hotswap, F.Cu at (76.2, 73.8)
- added SW32: SW_SPST, MX_Only:MXOnly-1U-Hotswap, F.Cu at (305.9, 218.7)
- added SW33: SW_SPST, MX_Only:MXOnly-1U-Hotswap, F.Cu at (95.2, 0.00)
- added SW34: SW_SPST, MX_Only:MXOnly-1U-Hotswap, F.Cu at (95.2, 19.1)
- added SW35: SW_SPST, MX_Only:MXOnly-1U-Hotswap, F.Cu at (95.2, 38.1)
- added SW36: SW_SPST, MX_Only:MXOnly-1U-Hotswap, F.Cu at (95.2, 57.1)
- added SW37: SW_SPST, MX_Only:MXOnly-1U-Hotswap, F.Cu at (95.2, 76.2)
- added SW38: SW_SPDT, Button_Switch_SMD:SW_SPDT_PCM12, B.Cu at (532.8, -9.01)
- added SW39: SW_SPST, MX_Only:MXOnly-1U-Hotswap, F.Cu at (95.2, 95.2)
- added SW4: SW_SPST, MX_Only:MXOnly-1U-Hotswap, F.Cu at (0.00, 19.1)
- added SW40: SW_SPST, MX_Only:MXOnly-1U-Hotswap, F.Cu at (346.3, 158.1)
- added SW41: SW_SPST, MX_Only:MXOnly-1U-Hotswap, F.Cu at (114.3, 9.53)
- added SW42: SW_SPST, MX_Only:MXOnly-1.25U-Hotswap, F.Cu at (114.3, 31.0)
- added SW43: SW_SPST, MX_Only:MXOnly-1.75U-Hotswap, F.Cu at (114.3, 59.5)
- added SW44: SW_SPST, MX_Only:MXOnly-1.5U-Hotswap, F.Cu at (114.3, 90.5)
- added SW45: SW_SPST, MX_Only:MXOnly-1U-Hotswap, F.Cu at (386.6, 97.5)
- added SW46: Rotary_Encoder_Switch, Rotary_Encoder:RotaryEncoder_Alps_EC11E-Switch_Vertical_H20mm, F.Cu at (365.1, 42.1)
- added SW47: SW_SPDT, Button_Switch_SMD:SW_SPDT_PCM12, B.Cu at (522.9, -9.01)
- added SW48: SW_SPST, MX_Only:MXOnly-1U-Hotswap, F.Cu at (152.4, 9.53)
- added SW49: SW_SPST, MX_Only:MXOnly-1U-Hotswap, F.Cu at (152.4, 28.6)
- added SW5: SW_SPST, MX_Only:MXOnly-1U-Hotswap, F.Cu at (0.00, 38.1)
- added SW50: SW_SPST, MX_Only:MXOnly-1.5U-Hotswap, F.Cu at (152.4, 52.4)
- added SW51: SW_SPST, MX_Only:MXOnly-2U-Hotswap-VerticalStabilizers, F.Cu at (152.4, 85.7)
- added SW52: SW_SPST, MX_Only:MXOnly-1U-Hotswap, F.Cu at (366.5, 117.7)
- added SW53: SW_SPST, MX_Only:MXOnly-1U-Hotswap, F.Cu at (171.4, 0.00)
- added SW54: SW_SPST, MX_Only:MXOnly-1U-Hotswap, F.Cu at (171.4, 19.1)
- added SW55: SW_SPST, MX_Only:MXOnly-1U-Hotswap, F.Cu at (171.4, 38.1)
- added SW56: SW_SPST, MX_Only:MXOnly-1U-Hotswap, F.Cu at (171.4, 57.1)
- added SW57: SW_SPST, MX_Only:MXOnly-1U-Hotswap, F.Cu at (171.4, 76.2)
- added SW58: SW_SPST, MX_Only:MXOnly-1U-Hotswap, F.Cu at (171.4, 95.2)
- added SW59: SW_SPST, MX_Only:MXOnly-1U-Hotswap, F.Cu at (285.7, 182.0)
- added SW6: SW_SPST, MX_Only:MXOnly-1U-Hotswap, F.Cu at (0.00, 57.1)
- added SW60: SW_SPST, MX_Only:MXOnly-1U-Hotswap, F.Cu at (346.2, 97.5)
- added SW61: SW_SPST, MX_Only:MXOnly-1U-Hotswap, F.Cu at (190.5, -2.38)
- added SW62: SW_SPST, MX_Only:MXOnly-1U-Hotswap, F.Cu at (190.5, 16.7)
- added SW63: SW_SPST, MX_Only:MXOnly-1U-Hotswap, F.Cu at (190.5, 35.7)
- added SW64: SW_SPST, MX_Only:MXOnly-1U-Hotswap, F.Cu at (190.5, 54.8)
- added SW65: SW_SPST, MX_Only:MXOnly-1U-Hotswap, F.Cu at (190.5, 73.8)
- added SW67: SW_SPST, MX_Only:MXOnly-1U-Hotswap, F.Cu at (346.2, 77.3)
- added SW68: SW_SPST, MX_Only:MXOnly-1U-Hotswap, F.Cu at (209.6, -4.76)
- added SW69: SW_SPST, MX_Only:MXOnly-1U-Hotswap, F.Cu at (209.6, 14.3)
- added SW7: SW_SPST, MX_Only:MXOnly-1U-Hotswap, F.Cu at (0.00, 76.2)
- added SW70: SW_SPST, MX_Only:MXOnly-1U-Hotswap, F.Cu at (209.6, 33.3)
- added SW71: SW_SPST, MX_Only:MXOnly-1U-Hotswap, F.Cu at (209.6, 52.4)
- added SW72: SW_SPST, MX_Only:MXOnly-1U-Hotswap, F.Cu at (209.6, 71.4)
- added SW73: SW_SPST, MX_Only:MXOnly-2.75U-Hotswap-ReversedStabilizers, F.Cu at (207.2, 92.9)
- added SW74: SW_SPST, MX_Only:MXOnly-1U-Hotswap, F.Cu at (228.6, -2.38)
- added SW75: SW_SPST, MX_Only:MXOnly-1U-Hotswap, F.Cu at (228.6, 16.7)
- added SW76: SW_SPST, MX_Only:MXOnly-1U-Hotswap, F.Cu at (228.6, 35.7)
- added SW77: SW_SPST, MX_Only:MXOnly-1U-Hotswap, F.Cu at (228.6, 54.8)
- added SW78: SW_SPST, MX_Only:MXOnly-1U-Hotswap, F.Cu at (228.6, 73.8)
- added SW79: SW_SPST, MX_Only:MXOnly-1U-Hotswap, F.Cu at (247.7, 0.00)
- added SW8: SW_SPST, MX_Only:MXOnly-1U-Hotswap, F.Cu at (449.7, 118.1)
- added SW80: SW_SPST, MX_Only:MXOnly-1U-Hotswap, F.Cu at (247.7, 19.1)
- added SW81: SW_SPST, MX_Only:MXOnly-1U-Hotswap, F.Cu at (247.7, 38.1)
- added SW82: SW_SPST, MX_Only:MXOnly-1U-Hotswap, F.Cu at (247.7, 57.1)
- added SW83: SW_SPST, MX_Only:MXOnly-1U-Hotswap, F.Cu at (247.7, 76.2)
- added SW84: SW_SPST, MX_Only:MXOnly-1U-Hotswap, F.Cu at (436.6, 42.1)
- added SW85: SW_SPST, MX_Only:MXOnly-1U-Hotswap, F.Cu at (266.7, 0.00)
- added SW86: SW_SPST, MX_Only:MXOnly-1U-Hotswap, F.Cu at (266.7, 19.1)
- added SW87: SW_SPST, MX_Only:MXOnly-1U-Hotswap, F.Cu at (266.7, 38.1)
- added SW88: SW_SPST, MX_Only:MXOnly-1U-Hotswap, F.Cu at (266.7, 57.1)
- added SW89: SW_SPST, MX_Only:MXOnly-1U-Hotswap, F.Cu at (266.7, 76.2)
- added SW9: SW_SPST, MX_Only:MXOnly-1U-Hotswap, F.Cu at (429.5, 138.3)
- added SW90: SW_SPST, MX_Only:MXOnly-1U-Hotswap, F.Cu at (386.7, 178.3)
- added SW91: SW_SPST, MX_Only:MXOnly-1U-Hotswap, F.Cu at (346.3, 198.5)
- added SW92: Rotary_Encoder_Switch, Rotary_Encoder:RotaryEncoder_Alps_EC11E-Switch_Vertical_H20mm, F.Cu at (287.6, 29.4)
- added U1: nRF52840_holyiot_18010, kicad-keyboard-parts:nRF52840_holyiot_18010, B.Cu at (247.7, 92.9)
- added U2: XC6206, Package_TO_SOT_SMD:SOT-23, B.Cu at (479.8, -82.3)
- added U3: TP4054, Package_TO_SOT_SMD:SOT-23-5, B.Cu at (517.5, -45.3)
- added U4: nRF52840_holyiot_18010, kicad-keyboard-parts:nRF52840_holyiot_18010, B.Cu at (19.1, 92.9)
- added U5: TP4054, Package_TO_SOT_SMD:SOT-23-5, B.Cu at (560.7, -1.46)
- added U6: XC6206, Package_TO_SOT_SMD:SOT-23, B.Cu at (500.0, -62.6)
- added USB1: HRO-TYPE-C-31-M-12, Type-C:HRO-TYPE-C-31-M-12-HandSoldering, B.Cu at (-11.1, 25.4)
- added USB2: HRO-TYPE-C-31-M-12, Type-C:HRO-TYPE-C-31-M-12-HandSoldering, B.Cu at (277.8, 25.4)
Routing:
- net RH_COL1: track 0.00 -> 109.9 mm, vias 0 -> 6
- net LH_COL5: track 0.00 -> 109.9 mm, vias 0 -> 6
- net RH_ROW4: track 0.00 -> 100.9 mm
- net RH_ROW3: track 0.00 -> 100.9 mm
- net LH_ROW4: track 0.00 -> 100.9 mm
- net LH_ROW3: track 0.00 -> 100.9 mm
- net LH_ROW1: track 0.00 -> 100.9 mm
- net LH_ROW0: track 0.00 -> 100.9 mm
- net RH_ROW2: track 0.00 -> 100.9 mm
- net RH_ROW0: track 0.00 -> 100.9 mm
- net LH_ROW2: track 0.00 -> 100.9 mm
- net RH_COL6: track 0.00 -> 88.4 mm, vias 0 -> 5
- net RH_COL5: track 0.00 -> 88.4 mm, vias 0 -> 5
- net RH_COL4: track 0.00 -> 88.4 mm, vias 0 -> 5
- net LH_COL4: track 0.00 -> 88.4 mm, vias 0 -> 5
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- removed copper zone on B.Cu, net GND
- removed copper zone on F.Cu, net GND

Commit message: Various commits
I can't remember exactly what's changed since last time, but this is the most recent version!
Parts:
- removed the REF** at (133.3, 61.9)
- added J10: Conn_01x05, Connector_JST:JST_SH_SM05B-SRSS-TB_1x05-1MP_P1.00mm_Horizontal, B.Cu at (148.6, 191.6)
- added J2: Conn_01x05, Connector_JST:JST_SH_SM05B-SRSS-TB_1x05-1MP_P1.00mm_Horizontal, B.Cu at (119.1, 199.2)
- added J3: Conn_01x05, Connector_JST:JST_SH_SM05B-SRSS-TB_1x05-1MP_P1.00mm_Horizontal, B.Cu at (119.1, 191.6)
- added J4: Conn_01x05, Connector_JST:JST_SH_SM05B-SRSS-TB_1x05-1MP_P1.00mm_Horizontal, B.Cu at (128.9, 199.2)
- added J5: Conn_01x05, Connector_JST:JST_SH_SM05B-SRSS-TB_1x05-1MP_P1.00mm_Horizontal, B.Cu at (128.9, 191.6)
- added J7: Conn_01x05, Connector_JST:JST_SH_SM05B-SRSS-TB_1x05-1MP_P1.00mm_Horizontal, B.Cu at (138.8, 199.2)
- added J8: Conn_01x05, Connector_JST:JST_SH_SM05B-SRSS-TB_1x05-1MP_P1.00mm_Horizontal, B.Cu at (138.8, 191.6)
- added J9: Conn_01x05, Connector_JST:JST_SH_SM05B-SRSS-TB_1x05-1MP_P1.00mm_Horizontal, B.Cu at (148.6, 199.2)
- added REF**: breakaway-mousebites, Keebio-Parts:breakaway-mousebites, F.Cu at (147.6, 109.5)
- added REF**: breakaway-mousebites, Keebio-Parts:breakaway-mousebites, F.Cu at (95.2, 8.73)
- added REF**: breakaway-mousebites, Keebio-Parts:breakaway-mousebites, F.Cu at (95.2, 11.1)
- added REF**: breakaway-mousebites, Keebio-Parts:breakaway-mousebites, F.Cu at (19.1, 11.1)
- added REF**: breakaway-mousebites, Keebio-Parts:breakaway-mousebites, F.Cu at (123.8, 34.9)
- added REF**: breakaway-mousebites, Keebio-Parts:breakaway-mousebites, F.Cu at (128.6, 34.9)
- added REF**: breakaway-mousebites, Keebio-Parts:breakaway-mousebites, F.Cu at (128.6, 88.9)
- added REF**: breakaway-mousebites, Keebio-Parts:breakaway-mousebites, F.Cu at (123.8, 88.9)
- added REF**: breakaway-mousebites, Keebio-Parts:breakaway-mousebites, F.Cu at (147.6, 104.8)
- added REF**: breakaway-mousebites, Keebio-Parts:breakaway-mousebites, F.Cu at (104.8, 104.8)
- added REF**: breakaway-mousebites, Keebio-Parts:breakaway-mousebites, F.Cu at (104.8, 109.5)
- added REF**: breakaway-mousebites, Keebio-Parts:breakaway-mousebites, F.Cu at (233.4, 11.1)
- added REF**: breakaway-mousebites, Keebio-Parts:breakaway-mousebites, F.Cu at (233.4, 8.73)
- added REF**: breakaway-mousebites, Keebio-Parts:breakaway-mousebites, F.Cu at (157.2, 11.1)
- added REF**: breakaway-mousebites, Keebio-Parts:breakaway-mousebites, F.Cu at (157.2, 8.73)
- added REF**: breakaway-mousebites, Keebio-Parts:breakaway-mousebites, F.Cu at (19.1, 8.73)
- added SW1: SW_SPST, Keebio-Parts:SW_SPST_TL3342, B.Cu at (139.7, 169.9)
- added SW66: SW_SPST, Keebio-Parts:SW_SPST_TL3342, B.Cu at (149.2, 169.9)
- J1, J6: moved to B.Cu
- SW32, SW40, SW45, SW84, SW90, SW91: footprint MX_Only:MXOnly-1U-Hotswap -> MX_Only:MXOnly-1.25U-Hotswap
- moved D2 586.1 mm to (-7.14, 162.7), turned to 90 degrees
- moved D9 548.5 mm to (11.9, 162.7), turned to 90 degrees
- moved D15 537.1 mm to (31.0, 162.7), turned to 90 degrees
- moved D8 505.4 mm to (11.9, 143.7), turned to 90 degrees
- moved SW8 441.7 mm to (8.73, 143.7)
- moved SW2 439.8 mm to (-10.3, 162.7)
- moved SW15 426.8 mm to (27.8, 162.7)
- moved SW9 421.4 mm to (8.73, 162.7)
- moved D91 413.7 mm to (157.2, 118.3), turned to 180 degrees
- moved D85 412.0 mm to (138.1, 118.3), turned to 180 degrees
- moved D92 390.1 mm to (181.8, 116.7), turned to 90 degrees
- moved D53 344.9 mm to (269.9, 202.4), turned to 90 degrees
- moved D62 331.6 mm to (288.9, 202.4), turned to 90 degrees
- moved D68 314.4 mm to (308.0, 202.4), turned to 90 degrees
- moved SW84 308.8 mm to (138.1, 121.4), turned to 90 degrees
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Routing:
- net RH_ROW1: track 0.00 -> 88.6 mm
- net DB2_ROW0_B: track 0.00 -> 58.3 mm
- net DB_COL1: track 0.00 -> 51.8 mm, vias 0 -> 2
- net DB_COL1_B: track 0.00 -> 51.8 mm, vias 0 -> 2
- net DB2_ROW0: track 0.00 -> 43.0 mm
- net DB_ROW0_B: track 0.00 -> 28.1 mm
- net DB_ROW0: track 0.00 -> 28.1 mm
- net DB_COL0_B: track 0.00 -> 23.9 mm, vias 0 -> 2
- net DB_COL0: track 0.00 -> 23.9 mm, vias 0 -> 2
- net DB_ROW1_B: track 0.00 -> 19.6 mm
- net DB_ROW1: track 0.00 -> 19.6 mm
- net LH_COL2: track 88.4 -> 69.3 mm
- net LH_COL1: track 88.4 -> 69.3 mm
- net LH_COL0: track 88.4 -> 69.3 mm
- net LH_COL3: track 88.4 -> 69.3 mm
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Other:
- board outline added: 271.5 x 147.6 mm

Commit message: Various changes, finished placing switches
Parts:
- added REF**: breakaway-mousebites, Keebio-Parts:breakaway-mousebites, F.Cu at (19.1, 102.4)
- added REF**: breakaway-mousebites, Keebio-Parts:breakaway-mousebites, F.Cu at (19.1, 107.2)
- added REF**: breakaway-mousebites, Keebio-Parts:breakaway-mousebites, F.Cu at (233.4, 102.4)
- added REF**: breakaway-mousebites, Keebio-Parts:breakaway-mousebites, F.Cu at (233.4, 107.2)
- C1: moved to B.Cu
- SW46, SW92: footprint Rotary_Encoder:RotaryEncoder_Alps_EC11E-Switch_Vertical_H20mm -> Keebio-Parts:RotaryEncoder_Alps_EC11E-Switch_Vertical_H20mm
- moved D40 552.2 mm to (0.79, 25.4), turned to 90 degrees
- moved C1 339.7 mm to (546.9, 6.35)
- moved D47 288.3 mm to (250.8, 25.4), turned to 270 degrees
- moved SW46 196.6 mm to (114.3, 31.0), turned to 180 degrees
- moved SW92 135.2 mm to (138.1, 28.6), turned to 270 degrees
- moved J9 85.8 mm to (145.3, 113.5)
- moved D53 84.3 mm to (218.3, 135.7)
- moved D62 84.3 mm to (237.3, 135.7)
- moved D68 84.3 mm to (256.4, 135.7)
- moved SW52 84.3 mm to (215.1, 135.7)
- moved SW60 84.3 mm to (234.2, 135.7)
- moved SW67 84.3 mm to (253.2, 135.7)
- moved D61 84.3 mm to (237.3, 116.7)
- moved SW59 84.3 mm to (234.2, 116.7)
- moved D15 28.9 mm to (41.3, 135.7)
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Routing:
- net ENC_P2_B: track 0.00 -> 17.7 mm
- net ENC_P1_B: track 0.00 -> 11.4 mm
Other:
- board size 271.5 x 147.6 mm -> 272.3 x 159.5 mm

Commit message: Place components in new arrangement
Parts:
- removed the R3 at (464.0, -101.7)
- removed the REF** at (19.1, 102.4)
- removed the REF** at (19.1, 107.2)
- added R3: 10k, Resistor_SMD:R_0805_2012Metric, F.Cu at (250.8, 82.5)
- added R3: 10k, Resistor_SMD:R_0805_2012Metric, B.Cu at (1.59, 82.5)
- added REF**: breakaway-mousebites, Keebio-Parts:breakaway-mousebites, F.Cu at (19.1, 85.7)
- added REF**: breakaway-mousebites, Keebio-Parts:breakaway-mousebites, F.Cu at (19.1, 91.3)
- U1, U4: footprint kicad-keyboard-parts:nRF52840_holyiot_18010 -> kicad-keyboard-parts:nRF52840_holyiot_18010_HS_simple
- moved R9 563.9 mm to (-34.9, 119.1), turned to 180 degrees
- moved D39 556.0 mm to (-34.9, 121.4), turned to 180 degrees
- moved SW38 545.4 mm to (-4.76, 83.3), turned to 180 degrees
- moved U3 528.4 mm to (4.76, 82.5), turned to 180 degrees
- moved C1 524.7 mm to (27.8, 82.5), turned to 90 degrees
- moved C3 521.4 mm to (20.6, 82.5), turned to 270 degrees
- moved R7 504.9 mm to (25.4, 82.5), turned to 270 degrees
- moved D1 503.5 mm to (11.9, 82.5), turned to 90 degrees
- moved R5 499.9 mm to (0.79, 22.2), turned to 180 degrees
- moved F1 492.5 mm to (28.6, 64.3)
- moved C2 491.1 mm to (8.73, 19.8), turned to 180 degrees
- moved U2 490.9 mm to (17.5, 82.5), turned to 270 degrees
- moved Q1 487.4 mm to (8.73, 82.5), turned to 270 degrees
- moved R6 475.7 mm to (8.73, 17.5), turned to 180 degrees
- moved C4 475.5 mm to (14.3, 82.5), turned to 270 degrees
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Connections:
- D15 pad 1: DB_ROW1 -> DB1_ROW1
- D2 pad 1: DB_ROW0 -> DB1_ROW0
- D8 pad 1: DB_ROW0 -> DB1_ROW0
- D9 pad 1: DB_ROW1 -> DB1_ROW1
- R13 pad 1: BVOLT -> BVOLT_B
- R13 pad 2: VBAT -> VBAT_B
- R15 pad 1: GND -> GND1
- R15 pad 2: BVOLT -> BVOLT_B
- SW15 pad 1: DB_COL1 -> DB1_COL1
- SW2 pad 1: DB_COL1 -> DB1_COL1
- SW8 pad 1: DB_COL0 -> DB1_COL0
- SW9 pad 1: DB_COL0 -> DB1_COL0
Routing:
- net DB_COL1: track 51.8 -> 0.00 mm, vias 2 -> 0
- net DB1_COL1: track 0.00 -> 51.8 mm, vias 0 -> 2
- net DB1_ROW0: track 0.00 -> 30.0 mm
- net DB_ROW0: track 28.1 -> 0.00 mm
- net DB_COL0: track 23.9 -> 0.00 mm, vias 2 -> 0
- net DB1_COL0: track 0.00 -> 20.2 mm
- net DB_ROW1: track 19.6 -> 0.00 mm
- net DB1_ROW1: track 0.00 -> 19.6 mm
- net Net-(C7-Pad1): track 0.00 -> 12.8 mm
- net Net-(C4-Pad1): track 0.00 -> 12.2 mm
- net VBUS: track 0.00 -> 11.0 mm
- net VBUS_B: track 0.00 -> 9.18 mm
- net VBAT_B: track 0.00 -> 6.07 mm
- net DB_ROW0_B: track 28.1 -> 33.5 mm
- net VBAT: track 0.00 -> 5.29 mm
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Other:
- board size 272.3 x 159.5 mm -> 271.5 x 147.6 mm

Commit message: Further placement of parts
Parts:
- removed the R3 at (250.8, 82.5)
- moved J7 166.1 mm to (233.4, 62.7), turned to 180 degrees
- moved J8 135.6 mm to (233.4, 94.5)
- moved J4 124.4 mm to (88.1, 81.8), turned to 180 degrees
- moved J10 111.0 mm to (164.3, 81.8), turned to 180 degrees
- moved J5 88.1 mm to (88.1, 113.5)
- moved R2 19.2 mm to (9.53, 69.1)
- moved F1 19.2 mm to (9.53, 66.7)
- moved J9 19.1 mm to (164.3, 113.5)
- moved J3 18.3 mm to (19.1, 62.7)
- moved D44 14.1 mm to (114.3, 62.7)
Connections:
- D53 pad 1: DB_ROW0_B -> DB1_ROW0_B
- D61 pad 1: DB_ROW0_B -> DB1_ROW0_B
- D62 pad 1: DB_ROW1_B -> DB1_ROW1_B
- D68 pad 1: DB_ROW1_B -> DB1_ROW1_B
- SW52 pad 1: DB_COL1_B -> DB1_COL1_B
- SW59 pad 1: DB_COL0_B -> DB1_COL0_B
- SW60 pad 1: DB_COL0_B -> DB1_COL0_B
- SW67 pad 1: DB_COL1_B -> DB1_COL1_B
- SW73 pad 1: RH_COL4 -> RH_COL3
- USB2 pad 1: GND -> GND1
- USB2 pad 2: RAW -> RAW_B
Routing:
- net DB_COL1_B: track 51.8 -> 0.00 mm, vias 2 -> 0
- net DB1_COL1_B: track 0.00 -> 51.8 mm, vias 0 -> 2
- net DB_ROW0_B: track 33.5 -> 0.00 mm
- net DB1_ROW0_B: track 0.00 -> 33.5 mm
- net LH_COL3: track 69.3 -> 96.2 mm, vias 5 -> 6
- net RH_COL3: track 88.4 -> 113.3 mm, vias 5 -> 6
- net DB_COL0_B: track 20.2 -> 0.00 mm
- net DB1_COL0_B: track 0.00 -> 20.2 mm
- net DB_ROW1_B: track 19.6 -> 0.00 mm
- net DB1_ROW1_B: track 0.00 -> 19.6 mm
- net VBUS: track 11.0 -> 25.4 mm, vias 0 -> 2
- net Net-(D38-Pad2): track 0.00 -> 4.53 mm
- net Net-(D44-Pad2): track 0.00 -> 4.53 mm

Commit message: USB wiring, etc...
Parts:
- moved R14 406.9 mm to (134.9, 103.2)
- moved F2 299.6 mm to (242.9, 66.7)
- moved R16 281.1 mm to (242.9, 69.1)
- moved R10 259.1 mm to (242.9, 23.0)
- moved D39 157.4 mm to (121.4, 103.2), turned to 0 degrees
- moved R9 153.2 mm to (117.5, 103.2)
- moved D48 147.0 mm to (131.0, 103.2), turned to 180 degrees
- moved C2 33.7 mm to (-23.8, 28.6)
- moved R6 33.7 mm to (-23.8, 26.2)
- moved R11 24.9 mm to (242.9, 27.8)
- moved D43 12.4 mm to (107.2, 37.3)
- moved R1 8.87 mm to (9.53, 27.8)
- moved R5 8.77 mm to (9.53, 23.0)
- moved D45 7.49 mm to (114.3, 93.7)
- moved D87 2.25 mm to (243.7, 19.8)
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Connections:
- D50 pad 1: RH_ROW1 -> RH_ROW2
Routing:
- net ENC_P1: track 0.00 -> 77.7 mm, vias 0 -> 2
- net RAW_B: track 0.00 -> 65.0 mm, vias 0 -> 2
- net LH_COL0: track 69.3 -> 129.2 mm
- net LH_ROW0: track 100.9 -> 135.9 mm
- net LH_COL2: track 69.3 -> 104.2 mm, vias 5 -> 6
- net LH_COL1: track 69.3 -> 96.3 mm, vias 5 -> 6
- net RH_ROW3: track 100.9 -> 126.0 mm
- net RH_ROW0: track 100.9 -> 124.7 mm
- net Net-(R5-Pad2): track 0.00 -> 20.2 mm, vias 0 -> 2
- net Net-(R11-Pad2): track 0.00 -> 20.2 mm, vias 0 -> 2
- net Net-(R1-Pad2): track 0.00 -> 19.2 mm, vias 0 -> 2
- net Net-(R10-Pad2): track 0.00 -> 19.2 mm, vias 0 -> 2
- net RAW: track 0.00 -> 19.1 mm
- net ENC_P2: track 0.00 -> 17.7 mm
- net RH_ROW2: track 100.9 -> 117.9 mm
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- added copper zone on B.Cu, net GND
- added copper zone on F.Cu, net GND
- added copper zone on B.Cu, net GND1
- added copper zone on F.Cu, net GND1
Other:
- net class power removed
- net class raw removed
- net class usb power added: clearance 0.2, trace_width 0.35, via_dia 0.8, via_drill 0.4

Commit message: More wiring.
Routing:
- net GND1: track 8.59 -> 17.3 mm
Changed lines of the file:
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@@
     (thickness 1.6)
     (drawings 161)
-    (tracks 850)
+    (tracks 854)
     (zones 0)
     (modules 250)
@@
   (segment (start 253.15625 28.625) (end 252.4125 29.36875) (width 0.25) (layer B.Cu) (net 7))
   (segment (start 255.33 28.625) (end 253.15625 28.625) (width 0.25) (layer B.Cu) (net 7))
+  (segment (start 248.44375 23.8125) (end 248.44375 22.225) (width 0.25) (layer F.Cu) (net 7))
+  (segment (start 243.168749 21.825001) (end 241.975 23.01875) (width 0.25) (layer B.Cu) (net 7))
+  (segment (start 248.043751 21.825001) (end 243.168749 21.825001) (width 0.25) (layer B.Cu) (net 7))
+  (segment (start 248.44375 22.225) (end 248.043751 21.825001) (width 0.25) (layer B.Cu) (net 7))
   (segment (start 226.975 83.5) (end 227.0125 83.4625) (width 0.25) (layer B.Cu) (net 8))
   (segment (start 224.63125 83.5) (end 226.975 83.5) (width 0.25) (layer B.Cu) (net 8))
