File: pcbfiles/pcb.kicad_pcb (KiCad board)
At the start: 2 copper layers, 269.9 x 139.7 mm, 256 parts, among them J1 Conn_01x06, J2 Conn_01x06, J3 Conn_01x06, J4 Conn_01x06, J5 Conn_01x04_Female, J6 Conn_01x04_Female, Q1 AO3401A, Q2 AO3401A, SW1 SW_SPST, SW10 SW_SPST, SW11 SW_SPST, SW12 SW_SPST, SW13 SW_SPST, SW14 SW_SPST, SW15 SW_SPST, SW16 SW_SPST, SW17 SW_SPST, SW18 SW_SPST, SW19 SW_SPST, SW2 SW_SPST, SW20 SW_SPST, SW21 SW_SPST, SW22 SW_SPST, SW23 SW_SPST, SW24 SW_SPST, SW25 SW_SPST, SW26 SW_SPST, SW27 SW_SPST, SW28 SW_SPST, SW29 SW_SPST, SW3 SW_SPST, SW30 SW_SPST, SW31 SW_SPST, SW32 SW_SPST, SW33 SW_SPST, SW34 SW_SPST, SW35 SW_SPST, SW36 SW_SPST, SW37 SW_SPST, SW38 SW_SPST, SW39 SW_SPST, SW4 SW_SPST, SW40 SW_SPST, SW41 SW_SPST, SW42 SW_SPST, SW43 SW_SPST, SW44 SW_SPST, SW45 SW_SPST, SW46 SW_SPST, SW47 SW_SPST, SW48 SW_SPST, SW49 SW_SPST, SW5 SW_SPST, SW50 SW_SPST, SW51 SW_SPST, SW52 SW_SPST, SW53 SW_SPST, SW54 SW_SPST, SW55 SW_SPST, SW56 SW_SPST, SW57 SW_SPST, SW58 SW_SPST, SW59 SW_SPST, SW6 SW_SPST, SW60 SW_SPST, SW61 SW_SPST, SW62 SW_SPST, SW63 SW_SPST, SW64 SW_SPST, SW65 SW_SPST, SW66 SW_SPST, SW67 SW_SPST, SW68 SW_SPST, SW69 SW_SPST, SW7 SW_SPST, SW70 SW_SPST, SW71 SW_SPST, SW72 SW_SPST, SW73 SW_SPST, SW74 SW_SPST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

Commit message: Routing.
Connections:
- U5 pad 15: ENC_P1 -> unconnected-(U5-Pad15)
- U5 pad 16: ENC_A -> ENC_P1
- U5 pad 17: ENC_B -> ENC_A
- U5 pad 18: unconnected-(U5-Pad18) -> ENC_B
Routing:
- net ENC_P1: track 99.3 -> 255.2 mm, vias 5 -> 7
- net ENC_A: track 0.00 -> 149.1 mm, vias 0 -> 2
- net ENC_B: track 0.00 -> 146.5 mm, vias 0 -> 2
- net VBUS: track 93.3 -> 150.1 mm
- net DBA_P1: track 110.0 -> 157.8 mm
- net LH_COL4: track 199.0 -> 221.1 mm
- net DBA_P5: track 128.8 -> 115.9 mm
- net LH_COL5: track 168.8 -> 172.5 mm, vias 6 -> 7
- net DBA_P2: track 154.6 -> 153.7 mm
- net LH_COL3: track 179.1 -> 178.4 mm
- net GND: vias 1 -> 0

Commit message: Routing.
Routing:
- net VBUS: track 150.1 -> 252.7 mm, vias 2 -> 4
- net LH_COL3: track 178.4 -> 231.7 mm
- net DBA_P1: track 157.8 -> 201.4 mm
- net VBAT: track 27.2 -> 70.4 mm, vias 0 -> 2
- net DBA_P2: track 153.7 -> 194.9 mm
- net LH_COL4: track 221.1 -> 252.4 mm
- net LH_COL5: track 172.5 -> 197.2 mm
- net DBA_P3: track 119.7 -> 126.4 mm
- net Net-(C5-Pad1): track 8.79 -> 12.2 mm
- net DBA_P5: track 115.9 -> 119.0 mm
- net DBA_P6: track 114.9 -> 117.9 mm
- net DBA_P4: track 118.2 -> 120.3 mm

Commit message: Routing.
Connections:
- net Net-(J2-Pad1) renamed DBB_P1
- net Net-(J2-Pad2) renamed DBB_P2
- net Net-(J2-Pad3) renamed DBB_P3
- net Net-(J2-Pad4) renamed DBB_P4
- net Net-(J2-Pad5) renamed DBB_P5
- net Net-(J2-Pad6) renamed DBB_P6
Routing:
- net DBB_P2: track 0.00 -> 37.3 mm, vias 0 -> 1
- net DBB_P1: track 0.00 -> 37.3 mm, vias 0 -> 1
- net DBB_P6: track 0.00 -> 36.1 mm, vias 0 -> 1
- net DBB_P5: track 0.00 -> 33.7 mm, vias 0 -> 1
- net DBB_P3: track 0.00 -> 32.7 mm, vias 0 -> 1
- net DBB_P4: track 0.00 -> 31.8 mm, vias 0 -> 1

Commit message: Routing.
Parts:
- moved F1 47.6 mm to (270.5, 38.4)
- moved R4 47.6 mm to (272.9, 38.4)
Routing:
- net B_D-: track 5.37 -> 68.2 mm
- net B_D+: track 8.70 -> 68.4 mm
- net RAW_B: track 42.6 -> 17.9 mm
- net GND: track 23.8 -> 39.7 mm, vias 0 -> 5
- net RH_ROW2: vias 0 -> 2
Changed lines of the file:
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@@
   )
   (footprint "Resistor_SMD:R_0805_2012Metric" (layer "B.Cu")
-    (at 226.21875 47.625 90)
+    (at 272.9 38.3875 90)
     (descr "Resistor SMD 0805 (2012 Metric), square (rectangular) end terminal, IPC_7351 nominal, (Body size source: IPC-SM-782 page 72, https://www.pcb-3d.com/wordpress/wp-content/uploads/ipc-sm-782a_amendment_1_and_2.pdf), generated with kicad-footprint-generator")
     (tags "resistor")
@@
   )
   (footprint "Fuse:Fuse_1206_3216Metric" (layer "B.Cu")
-    (at 223.8375 47.625 90)
+    (at 270.51875 38.3875 90)
     (descr "Fuse SMD 1206 (3216 Metric), square (rectangular) end terminal, IPC_7351 nominal, (Body size source: http://www.tortai-tech.com/upload/download/2011102023233369053.pdf), generated with kicad-footprint-generator")
     (tags "fuse")
@@
   (segment (start 86.725 49.00625) (end 85.725 48.00625) (width 0.25) (layer "F.Cu") (net 1))
   (segment (start 103.25625 49.00625) (end 86.725 49.00625) (width 0.25) (layer "F.Cu") (net 1))
+  (via (at 0.6 27.75) (size 0.8) (drill 0.4) (layers "F.Cu" "B.Cu") (net 1))
+  (via (at 19.05 22.225) (size 0.8) (drill 0.4) (layers "F.Cu" "B.Cu") (free) (net 1))
+  (via (at 3.15125 32.85) (size 0.8) (drill 0.4) (layers "F.Cu" "B.Cu") (net 1))
+  (via (at 0.6 34.2) (size 0.8) (drill 0.4) (layers "F.Cu" "B.Cu") (net 1))
+  (via (at -7.14375 16.66875) (size 0.8) (drill 0.4) (layers "F.Cu" "B.Cu") (free) (net 1))
   (segment (start 97.59375 70.8) (end 97.63125 70.7625) (width 0.25) (layer "B.Cu") (net 1))
   (segment (start -4.8 40.6) (end -4.7625 40.6375) (width 0.25) (layer "B.Cu") (net 1))
+  (segment (start 0.6 27.75) (end 0.6 27.4875) (width 0.25) (layer "B.Cu") (net 1))
   (segment (start 95.25 70.8) (end 97.59375 70.8) (width 0.25) (layer "B.Cu") (net 1))
   (segment (start -7.14375 40.6) (end -4.8 40.6) (width 0.25) (layer "B.Cu") (net 1))
+  (segment (start 0.1 34.975) (end -1.33 34.975) (width 0.25) (layer "B.Cu") (net 1))
+  (segment (start 0.6 34.475) (end 0.6 34.2) (width 0.25) (layer "B.Cu") (net 1))
   (segment (start 102.39375 68.9) (end 102.371992 68.9) (width 0.25) (layer "B.Cu") (net 1))
   (segment (start 95.5675 71.1175) (end 95.25 70.8) (width 0.25) (layer "B.Cu") (net 1))
+  (segment (start 1.1 26.9875) (end 9.81875 26.9875) (width 0.25) (layer "B.Cu") (net 1))
+  (segment (start 10.31875 27.9) (end 10.31875 27.4875) (width 0.25) (layer "B.Cu") (net 1))
+  (segment (start 0.6 28.025) (end 0.6 27.75) (width 0.25) (layer "B.Cu") (net 1))
   (segment (start 102.39375 68.9) (end 103.03125 68.9) (width 0.25) (layer "B.Cu") (net 1))
+  (segment (start 0.1 28.525) (end -1.33 28.525) (width 0.25) (layer "B.Cu") (net 1))
+  (arc (start 1.1 26.9875) (mid 0.746447 27.133947) (end 0.6 27.4875) (width 0.25) (layer "B.Cu") (net 1))
+  (arc (start 9.81875 26.9875) (mid 10.172303 27.133947) (end 10.31875 27.4875) (width 0.25) (layer "B.Cu") (net 1))
+  (arc (start 0.6 28.025) (mid 0.453553 28.378553) (end 0.1 28.525) (width 0.25) (layer "B.Cu") (net 1))
+  (arc (start 0.6 34.475) (mid 0.453553 34.828553) (end 0.1 34.975) (width 0.25) (layer "B.Cu") (net 1))
   (segment (start 84.009511 80.98) (end 84.009511 70.95) (width 0.25) (layer "F.Cu") (net 2))
   (segment (start 82.560489 72.55) (end 82.560489 80.98) (width 0.25) (layer "F.Cu") (net 2))
@@
   (segment (start 51.308 62.23) (end 51.308 59.8) (width 0.25) (layer "B.Cu") (net 53))
   (arc (start 51.308 59.8) (mid 51.600893 59.092893) (end 52.308 58.8) (width 0.25) (layer "B.Cu") (net 53))
-  (segment (start 224.325 32.85) (end 223.8375 33.3375) (width 0.35) (layer "B.Cu") (net 54))
   (segment (start 248.2875 32.85) (end 249.344607 33.907107) (width 0.35) (layer "B.Cu") (net 54))
   (segment (start 256.71875 33.705002) (end 255.000857 33.705002) (width 0.35) (layer "B.Cu") (net 54))
   (segment (start 253.884538 29.3) (end 252.94875 29.3) (width 0.35) (layer "B.Cu") (net 54))
-  (segment (start 248.2875 32.85) (end 224.325 32.85) (width 0.35) (layer "B.Cu") (net 54))
   (segment (start 256.71875 29.794998) (end 255.000857 29.794998) (width 0.35) (layer "B.Cu") (net 54))
   (segment (start 254.591645 29.592893) (end 254.647304 29.648552) (width 0.35) (layer "B.Cu") (net 54))
@@
   (arc (start 153.9875 -2) (mid 154.280393 -2.707107) (end 154.9875 -3) (width 0.25) (layer "B.Cu") (net 57))
   (arc (start 229.1875 -3) (mid 229.894607 -2.707107) (end 230.1875 -2) (width 0.25) (layer "B.Cu") (net 57))
+  (segment (start 222.25 35.1) (end 225.425 35.1) (width 0.25) (layer "F.Cu") (net 58))
+  (via (at 225.425 35.1) (size 0.8) (drill 0.4) (layers "F.Cu" "B.Cu") (net 58))
+  (via (at 222.25 35.1) (size 0.8) (drill 0.4) (layers "F.Cu" "B.Cu") (net 58))
   (segment (start 134.9375 36.45) (end 134.9375 36.1) (width 0.25) (layer "B.Cu") (net 58))
   (segment (start 174.0375 35.1) (end 191.0875 35.1) (width 0.25) (layer "B.Cu") (net 58))
@@
   (segment (start 154.9875 35.1) (end 172.0375 35.1) (width 0.25) (layer "B.Cu") (net 58))
   (segment (start 249.2375 36.45) (end 249.2375 36.1) (width 0.25) (layer "B.Cu") (net 58))
-  (segment (start 212.1375 35.1) (end 229.1875 35.1) (width 0.25) (layer "B.Cu") (net 58))
   (segment (start 193.0875 35.1) (end 210.1375 35.1) (width 0.25) (layer "B.Cu") (net 58))
   (segment (start 173.0375 36.45) (end 173.0375 36.1) (width 0.25) (layer "B.Cu") (net 58))
   (segment (start 211.1375 36.45) (end 211.1375 36.1) (width 0.25) (layer "B.Cu") (net 58))
+  (segment (start 222.25 35.1) (end 212.1375 35.1) (width 0.25) (layer "B.Cu") (net 58))
+  (segment (start 229.1875 35.1) (end 225.425 35.1) (width 0.25) (layer "B.Cu") (net 58))
   (segment (start 231.1875 35.1) (end 248.2375 35.1) (width 0.25) (layer "B.Cu") (net 58))
   (arc (start 248.2375 35.1) (mid 248.944607 35.392893) (end 249.2375 36.1) (width 0.25) (layer "B.Cu") (net 58))
@@
   (segment (start 168.11875 68.85) (end 169.000857 67.967893) (width 0.35) (layer "B.Cu") (net 72))
   (segment (start 167.615197 68.346447) (end 168.11875 68.85) (width 0.35) (layer "B.Cu") (net 72))
-  (segment (start 226.21875 48.5375) (end 224.325 48.5375) (width 0.35) (layer "B.Cu") (net 72))
+  (segment (start 272.9 39.3) (end 271.00625 39.3) (width 0.35) (layer "B.Cu") (net 72))
   (segment (start 169.707964 67.675) (end 172.498286 67.675) (width 0.35) (layer "B.Cu") (net 72))
-  (segment (start 224.325 48.5375) (end 223.8375 49.025) (width 0.35) (layer "B.Cu") (net 72))
+  (segment (start 271.00625 39.3) (end 270.51875 39.7875) (width 0.35) (layer "B.Cu") (net 72))
   (segment (start 173.205393 67.967893) (end 174.1375 68.9) (width 0.35) (layer "B.Cu") (net 72))
   (segment (start 165.89375 68.2) (end 167.261643 68.2) (width 0.35) (layer "B.Cu") (net 72))
@@
   (segment (start 259.4975 78.74) (end 259.4975 80.9625) (width 0.25) (layer "B.Cu") (net 129))
   (segment (start 259.4975 78.74) (end 259.4725 78.74) (width 0.25) (layer "B.Cu") (net 129))
+  (segment (start 224.0625 66.8) (end 224.0625 31.75) (width 0.2) (layer "B.Cu") (net 132))
+  (segment (start 224.0625 31.75) (end 248.673286 31.75) (width 0.2) (layer "B.Cu") (net 132))
   (segment (start 254.11875 31.5) (end 252.94875 31.5) (width 0.2) (layer "B.Cu") (net 132))
   (segment (start 252.94875 32.5) (end 250.5375 32.5) (width 0.2) (layer "B.Cu") (net 132))
@@
   (segment (start 250.5375 32.5) (end 250.1875 32.85) (width 0.2) (layer "B.Cu") (net 132))
   (segment (start 254.61875 32) (end 254.61875 32) (width 0.2) (layer "B.Cu") (net 132))
-  (arc (start 248.673286 31.75) (mid 249.055969 31.82612) (end 249.380393 32.042893) (width 0.2) (layer "B.Cu") (net 132))
   (arc (start 254.11875 32.5) (mid 254.472303 32.353553) (end 254.61875 32) (width 0.2) (layer "B.Cu") (net 132))
   (arc (start 254.11875 31.5) (mid 254.472303 31.646447) (end 254.61875 32) (width 0.2) (layer "B.Cu") (net 132))
+  (arc (start 248.673286 31.75) (mid 249.055969 31.82612) (end 249.380393 32.042893) (width 0.2) (layer "B.Cu") (net 132))
   (segment (start 251.27875 31.5) (end 251.27875 31.5) (width 0.2) (layer "B.Cu") (net 133))
   (segment (start 252.94875 31) (end 251.77875 31) (width 0.2) (layer "B.Cu") (net 133))
@@
   (segment (start 250.1875 30.65) (end 250.5375 31) (width 0.2) (layer "B.Cu") (net 133))
   (segment (start 252.94875 32) (end 251.77875 32) (width 0.2) (layer "B.Cu") (net 133))
+  (segment (start 223.6125 31.3) (end 223.6125 65.8) (width 0.2) (layer "B.Cu") (net 133))
   (segment (start 250.5375 31) (end 250.77875 31) (width 0.2) (layer "B.Cu") (net 133))
+  (segment (start 246.81875 31.3) (end 223.6125 31.3) (width 0.2) (layer "B.Cu") (net 133))
+  (segment (start 249.1875 29.65) (end 247.81875 29.65) (width 0.2) (layer "B.Cu") (net 133))
+  (segment (start 247.31875 30.15) (end 247.31875 30.8) (width 0.2) (layer "B.Cu") (net 133))
+  (arc (start 247.81875 29.65) (mid 247.465197 29.796447) (end 247.31875 30.15) (width 0.2) (layer "B.Cu") (net 133))
   (arc (start 251.27875 31.5) (mid 251.132303 31.146447) (end 250.77875 31) (width 0.2) (layer "B.Cu") (net 133))
   (arc (start 251.27875 31.5) (mid 251.425197 31.853553) (end 251.77875 32) (width 0.2) (layer "B.Cu") (net 133))
+  (arc (start 250.1875 30.65) (mid 249.894607 29.942893) (end 249.1875 29.65) (width 0.2) (layer "B.Cu") (net 133))
+  (arc (start 247.31875 30.8) (mid 247.172303 31.153553) (end 246.81875 31.3) (width 0.2) (layer "B.Cu") (net 133))
   (arc (start 251.77875 31) (mid 251.425197 31.146447) (end 251.27875 31.5) (width 0.2) (layer "B.Cu") (net 133))
   (segment (start 13.208 5.08) (end 13.208 2.65) (width 0.25) (layer "B.Cu") (net 134))

Commit message: Significant work on Routing.
right side!
Parts:
- moved F1 29.1 mm to (242.9, 47.6)
- moved R4 29.1 mm to (245.3, 47.6)
- turned D75 to 0 degrees
Connections:
- D82 pad 1: DBA_COL1 -> DBA_ROW1
- D83 pad 1: DBA_COL1 -> DBA_ROW1
- D84 pad 1: DBA_COL1 -> DBA_ROW1
- D85 pad 1: DBA_COL1 -> DBA_ROW1
- U6 pad 11: unconnected-(U6-Pad11) -> RH_COL1
- U6 pad 13: RH_ROW4 -> unconnected-(U6-Pad13)
- U6 pad 15: RH_COL4 -> unconnected-(U6-Pad15)
- U6 pad 16: RH_COL3 -> unconnected-(U6-Pad16)
- U6 pad 17: RH_COL2 -> unconnected-(U6-Pad17)
- U6 pad 18: RH_COL1 -> unconnected-(U6-Pad18)
- U6 pad 2: ENC_A_B -> unconnected-(U6-Pad2)
- U6 pad 20: RH_ROW3 -> unconnected-(U6-Pad20)
- U6 pad 26: unconnected-(U6-Pad26) -> RH_COL4
- U6 pad 28: unconnected-(U6-Pad28) -> RH_COL5
- U6 pad 29: unconnected-(U6-Pad29) -> RH_ROW4
- U6 pad 3: ENC_B_B -> unconnected-(U6-Pad3)
- U6 pad 30: RH_ROW2 -> unconnected-(U6-Pad30)
- U6 pad 33: RH_ROW0 -> unconnected-(U6-Pad33)
- U6 pad 34: RH_ROW1 -> unconnected-(U6-Pad34)
- U6 pad 35: RH_COL5 -> unconnected-(U6-Pad35)
- U6 pad 36: RH_COL6 -> unconnected-(U6-Pad36)
- U6 pad 4: ENC_P1_B -> unconnected-(U6-Pad4)
- U6 pad 6: RH_ROW5 -> unconnected-(U6-Pad6)
- U6 pad 7: RH_COL3 -> unconnected-(U6-Pad7)
Routing:
- net RESET_B: track 6.30 -> 111.1 mm
- net VDD_NRF_B: track 4.79 -> 90.4 mm, vias 0 -> 2
- net BVOLT_B: track 2.38 -> 81.1 mm, vias 0 -> 2
- net DBA_ROW0: track 5.63 -> 78.7 mm
- net SWD_B: track 0.00 -> 69.1 mm, vias 0 -> 1
- net RH_COL1: track 108.6 -> 177.0 mm
- net DBA_COL2: track 0.00 -> 68.3 mm, vias 0 -> 2
- net SWC_B: track 0.00 -> 66.2 mm
- net DBA_ROW1: track 0.00 -> 62.4 mm
- net DBA_COL0: track 0.00 -> 49.5 mm, vias 0 -> 2
- net DBA_COL3: track 0.00 -> 49.3 mm, vias 0 -> 2
- net unconnected-(U6-Pad34): track 0.00 -> 40.1 mm, vias 0 -> 1
- net unconnected-(U6-Pad35): track 0.00 -> 39.5 mm, vias 0 -> 1
- net RH_ROW4: track 104.1 -> 137.5 mm, vias 0 -> 4
- net RH_ROW5: track 0.00 -> 30.4 mm
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
Commit message: Routing.
Routing:
- net unconnected-(U6-Pad36): track 29.8 -> 80.6 mm
- net unconnected-(U6-Pad34): track 40.1 -> 50.0 mm
- net unconnected-(U6-Pad35): track 39.5 -> 48.8 mm
Changed lines of the file:
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@@
   (arc (start 237.5 92.7) (mid 236.792893 92.992893) (end 236.5 93.7) (width 0.25) (layer "F.Cu") (net 206))
   (segment (start 228.35 95.8) (end 226.75 95.8) (width 0.25) (layer "B.Cu") (net 206))
-  (segment (start 239.55 102.3) (end 251.9 102.3) (width 0.25) (layer "F.Cu") (net 207))
-  (segment (start 251.9 102.3) (end 251.9 92.5) (width 0.25) (layer "F.Cu") (net 207))
   (segment (start 236.5 101.3) (end 236.5 98.9) (width 0.25) (layer "F.Cu") (net 207))
+  (segment (start 251.9 93.7) (end 251.9 101.3) (width 0.25) (layer "F.Cu") (net 207))
+  (segment (start 245 92.7) (end 250.9 92.7) (width 0.25) (layer "F.Cu") (net 207))
   (segment (start 240.704521 102.3) (end 239.55 102.3) (width 0.25) (layer "F.Cu") (net 207))
   (segment (start 239.55 102.3) (end 237.5 102.3) (width 0.25) (layer "F.Cu") (net 207))
+  (segment (start 243 89.6) (end 243 90.7) (width 0.25) (layer "F.Cu") (net 207))
   (segment (start 234.5 96.9) (end 228.35 96.9) (width 0.25) (layer "F.Cu") (net 207))
+  (segment (start 250.9 102.3) (end 239.55 102.3) (width 0.25) (layer "F.Cu") (net 207))
   (via (at 228.35 96.9) (size 0.8) (drill 0.4) (layers "F.Cu" "B.Cu") (net 207))
   (arc (start 236.5 98.9) (mid 235.914214 97.485786) (end 234.5 96.9) (width 0.25) (layer "F.Cu") (net 207))
   (arc (start 236.5 101.3) (mid 236.792893 102.007107) (end 237.5 102.3) (width 0.25) (layer "F.Cu") (net 207))
+  (arc (start 245 92.7) (mid 243.585786 92.114214) (end 243 90.7) (width 0.25) (layer "F.Cu") (net 207))
+  (arc (start 251.9 101.3) (mid 251.607107 102.007107) (end 250.9 102.3) (width 0.25) (layer "F.Cu") (net 207))
+  (arc (start 250.9 92.7) (mid 251.607107 92.992893) (end 251.9 93.7) (width 0.25) (layer "F.Cu") (net 207))
   (segment (start 226.75 96.9) (end 228.35 96.9) (width 0.25) (layer "B.Cu") (net 207))
-  (segment (start 252.4 102.8) (end 252.4 92.3) (width 0.25) (layer "F.Cu") (net 208))
+  (segment (start 237.5 102.8) (end 250.9 102.8) (width 0.25) (layer "F.Cu") (net 208))
+  (segment (start 252.4 101.3) (end 252.4 93.7) (width 0.25) (layer "F.Cu") (net 208))
+  (segment (start 250.9 92.2) (end 245 92.2) (width 0.25) (layer "F.Cu") (net 208))
   (segment (start 228.35 98) (end 234.5 98) (width 0.25) (layer "F.Cu") (net 208))
-  (segment (start 252.3 102.8) (end 237.5 102.8) (width 0.25) (layer "F.Cu") (net 208))
   (segment (start 236 99.5) (end 236 101.3) (width 0.25) (layer "F.Cu") (net 208))
-  (segment (start 252.3 102.8) (end 252.4 102.8) (width 0.25) (layer "F.Cu") (net 208))
+  (segment (start 243.5 90.7) (end 243.5 89.85) (width 0.25) (layer "F.Cu") (net 208))
   (via (at 228.35 98) (size 0.8) (drill 0.4) (layers "F.Cu" "B.Cu") (net 208))
+  (arc (start 250.9 102.8) (mid 251.96066 102.36066) (end 252.4 101.3) (width 0.25) (layer "F.Cu") (net 208))
+  (arc (start 245 92.2) (mid 243.93934 91.76066) (end 243.5 90.7) (width 0.25) (layer "F.Cu") (net 208))
+  (arc (start 252.4 93.7) (mid 251.96066 92.63934) (end 250.9 92.2) (width 0.25) (layer "F.Cu") (net 208))
   (arc (start 236 101.3) (mid 236.43934 102.36066) (end 237.5 102.8) (width 0.25) (layer "F.Cu") (net 208))
-  (arc (start 236 99.5) (mid 235.56066 98.43934) (end 234.5 98) (width 0.25) (layer "F.Cu") (net 208))
+  (arc (start 234.5 98) (mid 235.56066 98.43934) (end 236 99.5) (width 0.25) (layer "F.Cu") (net 208))
   (segment (start 226.75 98) (end 228.35 98) (width 0.25) (layer "B.Cu") (net 208))
   (segment (start 53.975 115.825) (end 53.975 115.475) (width 0.25) (layer "B.Cu") (net 209))
@@
   (via (at 211.65 98) (size 0.8) (drill 0.4) (layers "F.Cu" "B.Cu") (net 211))
   (segment (start 213.25 98) (end 211.65 98) (width 0.25) (layer "B.Cu") (net 211))
-  (segment (start 252.9 103.3) (end 252.9 102.4) (width 0.25) (layer "F.Cu") (net 212))
-  (segment (start 235.5 100.1) (end 235.5 101.3) (width 0.25) (layer "F.Cu") (net 212))
-  (segment (start 228.35 99.1) (end 234.5 99.1) (width 0.25) (layer "F.Cu") (net 212))
-  (segment (start 237.5 103.3) (end 252.9 103.3) (width 0.25) (layer "F.Cu") (net 212))
+  (segment (start 259.04798 73.2) (end 244 73.2) (width 0.25) (layer "F.Cu") (net 212))
+  (segment (start 245 91.7) (end 250.9 91.7) (width 0.25) (layer "F.Cu") (net 212))
+  (segment (start 244 73.2) (end 244 90.7) (width 0.25) (layer "F.Cu") (net 212))
+  (segment (start 234.5 99.1) (end 228.35 99.1) (width 0.25) (layer "F.Cu") (net 212))
+  (segment (start 250.9 103.3) (end 237.5 103.3) (width 0.25) (layer "F.Cu") (net 212))
+  (segment (start 252.9 93.7) (end 252.9 101.3) (width 0.25) (layer "F.Cu") (net 212))
+  (segment (start 235.5 101.3) (end 235.5 100.1) (width 0.25) (layer "F.Cu") (net 212))
   (via (at 228.35 99.1) (size 0.8) (drill 0.4) (layers "F.Cu" "B.Cu") (free) (net 212))
   (arc (start 237.5 103.3) (mid 236.085786 102.714214) (end 235.5 101.3) (width 0.25) (layer "F.Cu") (net 212))
-  (arc (start 234.5 99.1) (mid 235.207107 99.392893) (end 235.5 100.1) (width 0.25) (layer "F.Cu") (net 212))
+  (arc (start 250.9 103.3) (mid 252.314214 102.714214) (end 252.9 101.3) (width 0.25) (layer "F.Cu") (net 212))
+  (arc (start 235.5 100.1) (mid 235.207107 99.392893) (end 234.5 99.1) (width 0.25) (layer "F.Cu") (net 212))
+  (arc (start 244 90.7) (mid 244.292893 91.407107) (end 245 91.7) (width 0.25) (layer "F.Cu") (net 212))
+  (arc (start 252.9 93.7) (mid 252.314214 92.285786) (end 250.9 91.7) (width 0.25) (layer "F.Cu") (net 212))
   (segment (start 226.75 99.1) (end 228.35 99.1) (width 0.25) (layer "B.Cu") (net 212))
   (segment (start 229.064214 92.2) (end 241.2 92.2) (width 0.25) (layer "F.Cu") (net 214))

Commit message: Routing
Connections:
- U6 pad 30: unconnected-(U6-Pad30) -> RH_COL4
- U6 pad 33: unconnected-(U6-Pad33) -> RH_ROW1
- U6 pad 34: unconnected-(U6-Pad34) -> RH_ROW2
- U6 pad 35: unconnected-(U6-Pad35) -> RH_ROW3
- U6 pad 36: unconnected-(U6-Pad36) -> RH_COL6
Routing:
- net RH_ROW2: track 124.9 -> 232.2 mm, vias 2 -> 4
- net RH_ROW1: track 111.4 -> 208.2 mm, vias 0 -> 2
- net RH_COL4: track 83.5 -> 173.7 mm, vias 6 -> 7
- net RH_ROW3: track 136.0 -> 223.9 mm, vias 4 -> 6
- net unconnected-(U6-Pad36): track 80.6 -> 0.00 mm, vias 1 -> 0
- net RH_COL6: track 87.3 -> 167.4 mm, vias 5 -> 6
- net unconnected-(U6-Pad34): track 50.0 -> 0.00 mm, vias 1 -> 0
- net unconnected-(U6-Pad35): track 48.8 -> 0.00 mm, vias 1 -> 0
- net unconnected-(U6-Pad33): track 21.5 -> 0.00 mm, vias 1 -> 0
- net unconnected-(U6-Pad30): track 16.6 -> 0.00 mm, vias 1 -> 0
- net RAW_B: track 39.1 -> 36.3 mm

Commit message: Routing.
Connections:
- U6 pad 30: RH_COL4 -> RH_ROW0
Routing:
- net RH_ROW0: track 124.9 -> 236.3 mm, vias 0 -> 2
- net RH_COL6: track 167.4 -> 197.1 mm
- net RH_COL5: track 108.4 -> 131.7 mm
- net RH_COL4: track 173.7 -> 158.1 mm, vias 7 -> 6
- net LH_COL3: track 231.7 -> 230.7 mm
- net LH_COL4: track 252.4 -> 251.7 mm
