File: pcbfiles/pcb.sch (KiCad schematic (older format))
At the start: 54 parts, among them J1 Conn_01x04_Female, Q1 AO3401A, SW1 SW_SPST, SW38 SW_SPDT, U2 XC6206, U3 TP4054, U4 nRF52840_holyiot_18010

Commit message: continue schematic, test pcb idea
Parts:
- added D? (x43): D_Small, symbol Device:D_Small
- added J?: Conn_01x05, symbol Connector_Generic:Conn_01x05
- added SW? (x43): SW_SPST, symbol Switch:SW_SPST
- added SW?: Rotary_Encoder_Switch, symbol Device:Rotary_Encoder_Switch
Connections:
- net labels added: DB_COL0, DB_COL1, DB_ROW0, DB_ROW1, ENC_A, ENC_B, ENC_P1, ENC_P2
- wire segments 114 -> 193

Commit message: PCB Layout, Diodes, Matrix
Main body switches placed, some parts of matrix routed, PCB progress.
Parts:
- added D49, D50, D51, D52, D53, D54, D55, D56, D57, D58, D59, D61, D62, D63, D64, D65, D66, D67, D68, D69, D70, D71, D72, D73, D74, D75, D76, D77, D78, D79, D80, D81, D82, D83, D84, D85, D86, D87, D88, D89, D90, D91, D92: D_Small, Diode_SMD:D_SOD-123, symbol Device:D_Small
- added J10, J3, J4, J5, J7, J8, J9: Conn_01x05, symbol Connector_Generic:Conn_01x05
- added SW48, SW49, SW52, SW53, SW54, SW55, SW56, SW57, SW58, SW59, SW60, SW61, SW62, SW63, SW64, SW65, SW67, SW68, SW69, SW70, SW71, SW72, SW74, SW75, SW76, SW77, SW78, SW79, SW80, SW81, SW82, SW83, SW84, SW85, SW86, SW87, SW88, SW89, SW90, SW91: SW_SPST, MX_Only:MXOnly-1U-Hotswap, symbol Switch:SW_SPST
- added SW50: SW_SPST, MX_Only:MXOnly-1.5U-Hotswap, symbol Switch:SW_SPST
- added SW51: SW_SPST, MX_Only:MXOnly-2U-Hotswap-VerticalStabilizers, symbol Switch:SW_SPST
- added SW73: SW_SPST, MX_Only:MXOnly-2.75U-Hotswap-ReversedStabilizers, symbol Switch:SW_SPST
- added SW92: Rotary_Encoder_Switch, Rotary_Encoder:RotaryEncoder_Alps_EC11E-Switch_Vertical_H20mm, symbol Device:Rotary_Encoder_Switch
- D10, D11, D12, D13, D14, D15, D16, D17, D18, D19, D2, D20, D21, D22, D23, D24, D25, D26, D27, D28, D29, D3, D30, D31, D32, D33, D34, D35, D36, D37, D38, D4, D41, D42, D43, D44, D45, D46, D5, D6, D7, D8, D9: renamed from D?; footprint (none) -> Diode_SMD:D_SOD-123
- SW10, SW11, SW12, SW13, SW14, SW15, SW16, SW17, SW18, SW19, SW2, SW20, SW21, SW22, SW23, SW24, SW25, SW27, SW28, SW29, SW3, SW30, SW31, SW32, SW33, SW34, SW35, SW36, SW37, SW39, SW4, SW40, SW41, SW45, SW5, SW6, SW7, SW8, SW9: renamed from SW?; footprint (none) -> MX_Only:MXOnly-1U-Hotswap
- SW26: renamed from SW?; footprint (none) -> MX_Only:MXOnly-2.25U-Hotswap-ReversedStabilizers
- SW42: renamed from SW?; footprint (none) -> MX_Only:MXOnly-1.25U-Hotswap
- SW43: renamed from SW?; footprint (none) -> MX_Only:MXOnly-1.75U-Hotswap
- SW44: renamed from SW?; footprint (none) -> MX_Only:MXOnly-1.5U-Hotswap
- SW46: renamed from SW?; footprint (none) -> Rotary_Encoder:RotaryEncoder_Alps_EC11E-Switch_Vertical_H20mm
- U1: renamed from U?; footprint kicad-keyboard-parts:nRF52840_holyiot_18010_nounderpins -> kicad-keyboard-parts:nRF52840_holyiot_18010
- U4: footprint kicad-keyboard-parts:nRF52840_holyiot_18010_nounderpins -> kicad-keyboard-parts:nRF52840_holyiot_18010
- gave numbers to parts that had none: 27
Connections:
- net labels added: DB1_COL0, DB1_COL0_B, DB1_COL1, DB1_COL1_B, DB1_ROW0, DB1_ROW0_B, DB1_ROW1, DB1_ROW1_B, DB2_COL0, DB2_COL0_B, DB2_COL1, DB2_COL1_B, DB2_COL2, DB2_COL2_B, DB2_ROW0, DB2_ROW0_B, DB2_ROW_B, DB_COL0_B, DB_COL1_B, DB_ROW0_B, DB_ROW1_B, ENC_A_B, ENC_B_B, ENC_P1_B, ENC_P2_B, LH_COL0, LH_COL1, LH_COL2, LH_COL3, LH_COL4, LH_COL5, LH_COL6, LH_ROW0, LH_ROW1, LH_ROW2, LH_ROW3, LH_ROW4, LH_ROW5, RH_COL0, RH_COL1, RH_COL2, RH_COL3, RH_COL4, RH_COL5, RH_COL6, RH_ROW0, RH_ROW1, RH_ROW2, RH_ROW3, RH_ROW4, RH_ROW5
- wire segments 193 -> 275
Other:
- moved on the sheet: BT1, BT2, D15, D2, D32, D41, D46, D8, D9, J2, SW15, SW2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

Commit message: Various commits
I can't remember exactly what's changed since last time, but this is the most recent version!
Parts:
- J10, J2, J3, J4, J5, J7, J8, J9: footprint (none) -> Connector_JST:JST_SH_SM05B-SRSS-TB_1x05-1MP_P1.00mm_Horizontal
- SW32, SW40, SW45, SW84, SW90, SW91: footprint MX_Only:MXOnly-1U-Hotswap -> MX_Only:MXOnly-1.25U-Hotswap
Changed lines of the file:
@@
 F 0 "J2" V 6214 6762 50  0000 R CNN
 F 1 "Conn_01x05" V 6123 6762 50  0000 R CNN
-F 2 "" H 6250 7050 50  0001 C CNN
+F 2 "Connector_JST:JST_SH_SM05B-SRSS-TB_1x05-1MP_P1.00mm_Horizontal" H 6250 7050 50  0001 C CNN
 F 3 "~" H 6250 7050 50  0001 C CNN
 	1    6250 7050
@@
 F 0 "SW40" H 9650 8685 50  0000 C CNN
 F 1 "SW_SPST" H 9650 8594 50  0000 C CNN
-F 2 "MX_Only:MXOnly-1U-Hotswap" H 9650 8450 50  0001 C CNN
+F 2 "MX_Only:MXOnly-1.25U-Hotswap" H 9650 8450 50  0001 C CNN
 F 3 "~" H 9650 8450 50  0001 C CNN
 	1    9650 8450
@@
 F 0 "SW45" H 10350 8685 50  0000 C CNN
 F 1 "SW_SPST" H 10350 8594 50  0000 C CNN
-F 2 "MX_Only:MXOnly-1U-Hotswap" H 10350 8450 50  0001 C CNN
+F 2 "MX_Only:MXOnly-1.25U-Hotswap" H 10350 8450 50  0001 C CNN
 F 3 "~" H 10350 8450 50  0001 C CNN
 	1    10350 8450
@@
 F 0 "SW32" H 8950 8685 50  0000 C CNN
 F 1 "SW_SPST" H 8950 8594 50  0000 C CNN
-F 2 "MX_Only:MXOnly-1U-Hotswap" H 8950 8450 50  0001 C CNN
+F 2 "MX_Only:MXOnly-1.25U-Hotswap" H 8950 8450 50  0001 C CNN
 F 3 "~" H 8950 8450 50  0001 C CNN
 	1    8950 8450
@@
 F 0 "J3" V 6914 6762 50  0000 R CNN
 F 1 "Conn_01x05" V 6823 6762 50  0000 R CNN
-F 2 "" H 6950 7050 50  0001 C CNN
+F 2 "Connector_JST:JST_SH_SM05B-SRSS-TB_1x05-1MP_P1.00mm_Horizontal" H 6950 7050 50  0001 C CNN
 F 3 "~" H 6950 7050 50  0001 C CNN
 	1    6950 7050
@@
 F 0 "J4" V 9014 6762 50  0000 R CNN
 F 1 "Conn_01x05" V 8923 6762 50  0000 R CNN
-F 2 "" H 9050 7050 50  0001 C CNN
+F 2 "Connector_JST:JST_SH_SM05B-SRSS-TB_1x05-1MP_P1.00mm_Horizontal" H 9050 7050 50  0001 C CNN
 F 3 "~" H 9050 7050 50  0001 C CNN
 	1    9050 7050
@@
 F 0 "J5" V 9714 6762 50  0000 R CNN
 F 1 "Conn_01x05" V 9623 6762 50  0000 R CNN
-F 2 "" H 9750 7050 50  0001 C CNN
+F 2 "Connector_JST:JST_SH_SM05B-SRSS-TB_1x05-1MP_P1.00mm_Horizontal" H 9750 7050 50  0001 C CNN
 F 3 "~" H 9750 7050 50  0001 C CNN
 	1    9750 7050
@@
 F 0 "J7" V 22414 6212 50  0000 R CNN
 F 1 "Conn_01x05" V 22323 6212 50  0000 R CNN
-F 2 "" H 22450 6500 50  0001 C CNN
+F 2 "Connector_JST:JST_SH_SM05B-SRSS-TB_1x05-1MP_P1.00mm_Horizontal" H 22450 6500 50  0001 C CNN
 F 3 "~" H 22450 6500 50  0001 C CNN
 	1    22450 6500
@@
 F 0 "SW90" H 26250 8135 50  0000 C CNN
 F 1 "SW_SPST" H 26250 8044 50  0000 C CNN
-F 2 "MX_Only:MXOnly-1U-Hotswap" H 26250 7900 50  0001 C CNN
+F 2 "MX_Only:MXOnly-1.25U-Hotswap" H 26250 7900 50  0001 C CNN
 F 3 "~" H 26250 7900 50  0001 C CNN
 	1    26250 7900
@@
 F 0 "SW91" H 26950 8135 50  0000 C CNN
 F 1 "SW_SPST" H 26950 8044 50  0000 C CNN
-F 2 "MX_Only:MXOnly-1U-Hotswap" H 26950 7900 50  0001 C CNN
+F 2 "MX_Only:MXOnly-1.25U-Hotswap" H 26950 7900 50  0001 C CNN
 F 3 "~" H 26950 7900 50  0001 C CNN
 	1    26950 7900
@@
 F 0 "SW84" H 25550 8135 50  0000 C CNN
 F 1 "SW_SPST" H 25550 8044 50  0000 C CNN
-F 2 "MX_Only:MXOnly-1U-Hotswap" H 25550 7900 50  0001 C CNN
+F 2 "MX_Only:MXOnly-1.25U-Hotswap" H 25550 7900 50  0001 C CNN
 F 3 "~" H 25550 7900 50  0001 C CNN
 	1    25550 7900
@@
 F 0 "J8" V 23114 6212 50  0000 R CNN
 F 1 "Conn_01x05" V 23023 6212 50  0000 R CNN
-F 2 "" H 23150 6500 50  0001 C CNN
+F 2 "Connector_JST:JST_SH_SM05B-SRSS-TB_1x05-1MP_P1.00mm_Horizontal" H 23150 6500 50  0001 C CNN
 F 3 "~" H 23150 6500 50  0001 C CNN
 	1    23150 6500
@@
 F 0 "J9" V 25614 6212 50  0000 R CNN
 F 1 "Conn_01x05" V 25523 6212 50  0000 R CNN
-F 2 "" H 25650 6500 50  0001 C CNN
+F 2 "Connector_JST:JST_SH_SM05B-SRSS-TB_1x05-1MP_P1.00mm_Horizontal" H 25650 6500 50  0001 C CNN
 F 3 "~" H 25650 6500 50  0001 C CNN
 	1    25650 6500
@@
 F 0 "J10" V 26314 6212 50  0000 R CNN
 F 1 "Conn_01x05" V 26223 6212 50  0000 R CNN
-F 2 "" H 26350 6500 50  0001 C CNN
+F 2 "Connector_JST:JST_SH_SM05B-SRSS-TB_1x05-1MP_P1.00mm_Horizontal" H 26350 6500 50  0001 C CNN
 F 3 "~" H 26350 6500 50  0001 C CNN
 	1    26350 6500

Commit message: Various changes, finished placing switches
Parts:
- SW46, SW92: footprint Rotary_Encoder:RotaryEncoder_Alps_EC11E-Switch_Vertical_H20mm -> Keebio-Parts:RotaryEncoder_Alps_EC11E-Switch_Vertical_H20mm
Changed lines of the file:
@@
 F 0 "SW46" V 10954 5230 50  0000 L CNN
 F 1 "Rotary_Encoder_Switch" V 11045 5230 50  0000 L CNN
-F 2 "Rotary_Encoder:RotaryEncoder_Alps_EC11E-Switch_Vertical_H20mm" H 10850 5160 50  0001 C CNN
+F 2 "Keebio-Parts:RotaryEncoder_Alps_EC11E-Switch_Vertical_H20mm" H 10850 5160 50  0001 C CNN
 F 3 "~" H 11000 5260 50  0001 C CNN
 	1    11000 5000
@@
 F 0 "SW92" V 27554 4680 50  0000 L CNN
 F 1 "Rotary_Encoder_Switch" V 27645 4680 50  0000 L CNN
-F 2 "Rotary_Encoder:RotaryEncoder_Alps_EC11E-Switch_Vertical_H20mm" H 27450 4610 50  0001 C CNN
+F 2 "Keebio-Parts:RotaryEncoder_Alps_EC11E-Switch_Vertical_H20mm" H 27450 4610 50  0001 C CNN
 F 3 "~" H 27600 4710 50  0001 C CNN
 	1    27600 4450

Commit message: Place components in new arrangement
Parts:
- U1, U4: footprint kicad-keyboard-parts:nRF52840_holyiot_18010 -> kicad-keyboard-parts:nRF52840_holyiot_18010_HS_simple
Connections:
- net DB_COL0 is gone; now on net DB1_COL0: SW8.1 (A), SW9.1 (A)
- net DB_COL1 is gone; now on net DB1_COL1: SW15.1 (A), SW2.1 (A)
- net DB_ROW0 is gone; now on net DB1_ROW0: D2.1 (K), D8.1 (K)
- net DB_ROW1 is gone; now on net DB1_ROW1: D15.1 (K), D9.1 (K)
- net BVOLT: no longer R13.1, R15.2
- net BVOLT_B: now also R13.1, R15.2
- net GND: no longer R15.1
- net GND1: now also R15.1
- net VBAT: no longer R13.2
- net VBAT_B: now also R13.2
Changed lines of the file:
@@
 F 0 "U4" H 1600 6365 50  0000 C CNN
 F 1 "nRF52840_holyiot_18010" H 1600 6274 50  0000 C CNN
-F 2 "kicad-keyboard-parts:nRF52840_holyiot_18010" H 1700 5250 50  0001 C CNN
+F 2 "kicad-keyboard-parts:nRF52840_holyiot_18010_HS_simple" H 1700 5250 50  0001 C CNN
 F 3 "http://www.holyiot.com/tp/2019042516322180424.pdf" H 1700 5250 50  0001 C CNN
 	1    1600 4850
@@
 F 0 "U1" H 17600 6365 50  0000 C CNN
 F 1 "nRF52840_holyiot_18010" H 17600 6274 50  0000 C CNN
-F 2 "kicad-keyboard-parts:nRF52840_holyiot_18010" H 17700 5250 50  0001 C CNN
+F 2 "kicad-keyboard-parts:nRF52840_holyiot_18010_HS_simple" H 17700 5250 50  0001 C CNN
 F 3 "http://www.holyiot.com/tp/2019042516322180424.pdf" H 17700 5250 50  0001 C CNN
 	1    17600 4850
@@
 	20350 1000 21000 1000
 Text GLabel 19950 2800 0    50   Input ~ 0
-VBAT
+VBAT_B
 $Comp
 L Device:R_Small R13
@@
 $EndComp
 $Comp
-L power:GND #PWR0114
+L power:GND1 #PWR0114
 U 1 1 6132A5F4
 P 21200 2800
 F 0 "#PWR0114" H 21200 2550 50  0001 C CNN
-F 1 "GND" V 21205 2672 50  0000 R CNN
+F 1 "GND1" V 21205 2672 50  0000 R CNN
 F 2 "" H 21200 2800 50  0001 C CNN
 F 3 "" H 21200 2800 50  0001 C CNN
@@
 	20350 2800 20500 2800
 Text GLabel 20500 3050 3    50   Input ~ 0
-BVOLT
+BVOLT_B
 Wire Wire Line
 	20500 2800 20500 3050
@@
 	5650 8900 5650 8550
 Text GLabel 6050 8750 0    50   Input ~ 0
-DB_ROW0
+DB1_ROW0
 Text GLabel 6750 8700 0    50   Input ~ 0
-DB_ROW1
+DB1_ROW1
 Text GLabel 6350 8100 0    50   Input ~ 0
-DB_COL0
+DB1_COL0
 Text GLabel 5650 8550 0    50   Input ~ 0
-DB_COL1
+DB1_COL1
 $Comp
 L Switch:SW_SPST SW40

Commit message: Further placement of parts
Connections:
- net DB_COL0_B is gone; now on net DB1_COL0_B: SW59.1 (A), SW60.1 (A)
- net DB_COL1_B is gone; now on net DB1_COL1_B: SW52.1 (A), SW67.1 (A)
- net DB_ROW0_B is gone; now on net DB1_ROW0_B: D53.1 (K), D61.1 (K)
- net DB_ROW1_B is gone; now on net DB1_ROW1_B: D62.1 (K), D68.1 (K)
- net GND: no longer USB2.1 (GND)
- net GND1: now also USB2.1 (GND)
- net RAW: no longer USB2.2 (VBUS)
- net RAW_B: now also USB2.2 (VBUS)
- net RH_COL3: now also SW73.1 (A)
- net RH_COL4: no longer SW73.1 (A)
Other:
- moved on the sheet: D74, SW73
Changed lines of the file:
@@
 $EndComp
 $Comp
-L power:GND #PWR0107
+L power:GND1 #PWR0107
 U 1 1 6132A54F
 P 17550 1050
 F 0 "#PWR0107" H 17550 800 50  0001 C CNN
-F 1 "GND" V 17555 922 50  0000 R CNN
+F 1 "GND1" V 17555 922 50  0000 R CNN
 F 2 "" H 17550 1050 50  0001 C CNN
 F 3 "" H 17550 1050 50  0001 C CNN
@@
 RAW_B
 Text GLabel 17550 1150 2    50   Input ~ 0
-RAW
+RAW_B
 Text GLabel 20000 1000 0    50   Input ~ 0
 RAW_B
@@
 L Switch:SW_SPST SW73
 U 1 1 6175E89F
-P 24200 5700
-F 0 "SW73" H 24200 5935 50  0000 C CNN
-F 1 "SW_SPST" H 24200 5844 50  0000 C CNN
-F 2 "MX_Only:MXOnly-2.75U-Hotswap-ReversedStabilizers" H 24200 5700 50  0001 C CNN
-F 3 "~" H 24200 5700 50  0001 C CNN
-	1    24200 5700
+P 23500 5700
+F 0 "SW73" H 23500 5935 50  0000 C CNN
+F 1 "SW_SPST" H 23500 5844 50  0000 C CNN
+F 2 "MX_Only:MXOnly-2.75U-Hotswap-ReversedStabilizers" H 23500 5700 50  0001 C CNN
+F 3 "~" H 23500 5700 50  0001 C CNN
+	1    23500 5700
 	1    0    0    -1
 $EndComp
@@
 L Device:D_Small D74
 U 1 1 6175E8A5
-P 24400 5800
-F 0 "D74" V 24446 5730 50  0000 R CNN
-F 1 "D_Small" V 24355 5730 50  0000 R CNN
-F 2 "Diode_SMD:D_SOD-123" V 24400 5800 50  0001 C CNN
-F 3 "~" V 24400 5800 50  0001 C CNN
-	1    24400 5800
+P 23700 5800
+F 0 "D74" V 23746 5730 50  0000 R CNN
+F 1 "D_Small" V 23655 5730 50  0000 R CNN
+F 2 "Diode_SMD:D_SOD-123" V 23700 5800 50  0001 C CNN
+F 3 "~" V 23700 5800 50  0001 C CNN
+	1    23700 5800
 	0    -1   -1   0
 $EndComp
@@
 	21900 5300 21900 5700
 Wire Wire Line
-	24000 5700 24000 5300
+	23300 5700 23300 5300
 Connection ~ 25400 3700
 Wire Wire Line
@@
 	21850 8350 21850 8000
 Text GLabel 22250 8200 0    50   Input ~ 0
-DB_ROW0_B
+DB1_ROW0_B
 Text GLabel 22950 8150 0    50   Input ~ 0
-DB_ROW1_B
+DB1_ROW1_B
 Text GLabel 22550 7550 0    50   Input ~ 0
-DB_COL0_B
+DB1_COL0_B
 Text GLabel 21850 8000 0    50   Input ~ 0
-DB_COL1_B
+DB1_COL1_B
 $Comp
 L Switch:SW_SPST SW90
@@
 	-1   0    0    1
 $EndComp
-Connection ~ 24000 5300
-Connection ~ 24400 5900
 Wire Wire Line
-	24400 5900 25800 5900
+	22300 5900 23700 5900
+Connection ~ 23300 5300
+Connection ~ 23700 5900
 Wire Wire Line
-	22300 5900 24400 5900
+	23700 5900 25800 5900
 $EndSCHEMATC

Commit message: USB wiring, etc...
Connections:
- net RH_ROW1: no longer D50.1 (K)
- net RH_ROW2: now also D50.1 (K)
Other:
- moved on the sheet: D50, SW49
Changed lines of the file:
@@
 L Switch:SW_SPST SW49
 U 1 1 6175E7EB
-P 21400 4100
-F 0 "SW49" H 21400 4335 50  0000 C CNN
-F 1 "SW_SPST" H 21400 4244 50  0000 C CNN
-F 2 "MX_Only:MXOnly-1U-Hotswap" H 21400 4100 50  0001 C CNN
-F 3 "~" H 21400 4100 50  0001 C CNN
-	1    21400 4100
+P 21400 4500
+F 0 "SW49" H 21400 4735 50  0000 C CNN
+F 1 "SW_SPST" H 21400 4644 50  0000 C CNN
+F 2 "MX_Only:MXOnly-1U-Hotswap" H 21400 4500 50  0001 C CNN
+F 3 "~" H 21400 4500 50  0001 C CNN
+	1    21400 4500
 	1    0    0    -1
 $EndComp
@@
 L Device:D_Small D50
 U 1 1 6175E7F1
-P 21600 4200
-F 0 "D50" V 21646 4130 50  0000 R CNN
-F 1 "D_Small" V 21555 4130 50  0000 R CNN
-F 2 "Diode_SMD:D_SOD-123" V 21600 4200 50  0001 C CNN
-F 3 "~" V 21600 4200 50  0001 C CNN
-	1    21600 4200
+P 21600 4600
+F 0 "D50" V 21646 4530 50  0000 R CNN
+F 1 "D_Small" V 21555 4530 50  0000 R CNN
+F 2 "Diode_SMD:D_SOD-123" V 21600 4600 50  0001 C CNN
+F 3 "~" V 21600 4600 50  0001 C CNN
+	1    21600 4600
 	0    -1   -1   0
 $EndComp
@@
 	0    -1   -1   0
 $EndComp
-Text GLabel 21600 4100 2    30   Input ~ 0
+Text GLabel 21600 4500 2    30   Input ~ 0
 ENC_P2_B
-Text GLabel 21200 4100 0    30   Input ~ 0
+Text GLabel 21200 4500 0    30   Input ~ 0
 ENC_P1_B
 $Comp
@@
 Wire Wire Line
 	25400 5300 25400 4900
-Wire Wire Line
-	21200 5700 21200 4900
-Connection ~ 21200 3700
 Wire Wire Line
 	21200 3700 21200 3300
@@
 	9200 5650 9900 5650
 Connection ~ 9200 5650
-Connection ~ 21200 4100
-Wire Wire Line
-	21200 4100 21200 3700
-Wire Wire Line
-	21200 4100 21200 4900
-Wire Wire Line
-	22300 4300 21600 4300
-Connection ~ 22300 4300
+Connection ~ 21200 4500
+Wire Wire Line
+	21200 4500 21200 4900
+Wire Wire Line
+	22300 4700 21600 4700
 Text GLabel 25400 3300 1    50   Input ~ 0
 RH_COL6
@@
 Wire Wire Line
 	23700 5900 25800 5900
+Connection ~ 22300 4700
+Wire Wire Line
+	21200 3700 21200 4500
+Wire Wire Line
+	21200 4900 21200 5700
+Connection ~ 21200 3700
 $EndSCHEMATC

Commit message: Various changes.
Connections:
- net GND: no longer J10.5 (Pin_5), J7.5 (Pin_5), J8.5 (Pin_5), J9.5 (Pin_5)
- net GND1: now also J10.5 (Pin_5), J7.5 (Pin_5), J8.5 (Pin_5), J9.5 (Pin_5)
- net D+_B renamed B_D+
- net D-_B renamed B_D-
Changed lines of the file:
@@
 	20000 1000 20150 1000
 Text GLabel 18000 6300 3    50   Input ~ 0
-D-_B
+B_D-
 Text GLabel 18100 6300 3    50   Input ~ 0
-D+_B
+B_D+
 $Comp
 L Battery_Management:MCP73831-3-OT U5
@@
 Connection ~ 18450 2100
 Text GLabel 18550 2100 2    50   Input ~ 0
-D+_B
+B_D+
 Text GLabel 18550 1100 2    50   Input ~ 0
-D-_B
+B_D-
 Wire Wire Line
 	23100 1450 23250 1450
@@
 DB1_ROW1_B
 $Comp
-L power:GND #PWR0131
+L power:GND1 #PWR0131
 U 1 1 6175E9BE
 P 22650 6700
 F 0 "#PWR0131" H 22650 6450 50  0001 C CNN
-F 1 "GND" H 22655 6527 50  0000 C CNN
+F 1 "GND1" H 22655 6527 50  0000 C CNN
 F 2 "" H 22650 6700 50  0001 C CNN
 F 3 "" H 22650 6700 50  0001 C CNN
@@
 $EndComp
 $Comp
-L power:GND #PWR0132
+L power:GND1 #PWR0132
 U 1 1 6175E9C4
 P 23350 6700
 F 0 "#PWR0132" H 23350 6450 50  0001 C CNN
-F 1 "GND" H 23355 6527 50  0000 C CNN
+F 1 "GND1" H 23355 6527 50  0000 C CNN
 F 2 "" H 23350 6700 50  0001 C CNN
 F 3 "" H 23350 6700 50  0001 C CNN
@@
 DB2_ROW_B
 $Comp
-L power:GND #PWR0133
+L power:GND1 #PWR0133
 U 1 1 6175E9D4
 P 25850 6700
 F 0 "#PWR0133" H 25850 6450 50  0001 C CNN
-F 1 "GND" H 25855 6527 50  0000 C CNN
+F 1 "GND1" H 25855 6527 50  0000 C CNN
 F 2 "" H 25850 6700 50  0001 C CNN
 F 3 "" H 25850 6700 50  0001 C CNN
@@
 DB2_ROW0_B
 $Comp
-L power:GND #PWR0134
+L power:GND1 #PWR0134
 U 1 1 6175E9E4
 P 26550 6700
 F 0 "#PWR0134" H 26550 6450 50  0001 C CNN
-F 1 "GND" H 26555 6527 50  0000 C CNN
+F 1 "GND1" H 26555 6527 50  0000 C CNN
 F 2 "" H 26550 6700 50  0001 C CNN
 F 3 "" H 26550 6700 50  0001 C CNN
