File: pcbfiles/plate.kicad_pcb (KiCad board)
At the start: 2 copper layers, 0 parts

Commit message: Almost there!
Parts:
- added REF**: MX_Cutout_1u, Keybage_MX_Cutout:MX_Cutout_1u, F.Cu at (76.2, 16.7)
- added REF**: MX_Cutout_1.25u, Keybage_MX_Cutout:MX_Cutout_1.25u, F.Cu at (114.3, 116.7)
- added REF**: MX_Cutout_2.25u, Keybage_MX_Cutout:MX_Cutout_2.25u, F.Cu at (64.3, 92.9)
- added REF**: MX_Cutout_1.25u, Keybage_MX_Cutout:MX_Cutout_1.25u, F.Cu at (114.3, 31.0)
- added REF**: MX_Cutout_1.75u, Keybage_MX_Cutout:MX_Cutout_1.75u, F.Cu at (114.3, 59.5)
- added REF**: MX_Cutout_1.5u, Keybage_MX_Cutout:MX_Cutout_1.5u, F.Cu at (114.3, 90.5)
- added REF**: MX_Cutout_1u, Keybage_MX_Cutout:MX_Cutout_1u, F.Cu at (95.2, 95.2)
- added REF**: MX_Cutout_1u, Keybage_MX_Cutout:MX_Cutout_1u, F.Cu at (114.3, 9.53)
- added REF**: MX_Cutout_1u, Keybage_MX_Cutout:MX_Cutout_1u, F.Cu at (95.2, 19.1)
- added REF**: MX_Cutout_1u, Keybage_MX_Cutout:MX_Cutout_1u, F.Cu at (95.2, 57.1)
- added REF**: MX_Cutout_1u, Keybage_MX_Cutout:MX_Cutout_1u, F.Cu at (95.2, 38.1)
- added REF**: MX_Cutout_1u, Keybage_MX_Cutout:MX_Cutout_1u, F.Cu at (38.1, 16.7)
- added REF**: MX_Cutout_1u, Keybage_MX_Cutout:MX_Cutout_1u, F.Cu at (95.2, 76.2)
- added REF**: MX_Cutout_1u, Keybage_MX_Cutout:MX_Cutout_1u, F.Cu at (95.2, 0.00)
- added REF**: MX_Cutout_1u, Keybage_MX_Cutout:MX_Cutout_1u, F.Cu at (76.2, 54.8)
- added REF**: MX_Cutout_1u, Keybage_MX_Cutout:MX_Cutout_1u, F.Cu at (76.2, 35.7)
- added REF**: MX_Cutout_1u, Keybage_MX_Cutout:MX_Cutout_1u, F.Cu at (76.2, 73.8)
- added REF**: MX_Cutout_1u, Keybage_MX_Cutout:MX_Cutout_1u, F.Cu at (76.2, -2.38)
- added REF**: MX_Cutout_1u, Keybage_MX_Cutout:MX_Cutout_1u, F.Cu at (57.1, 52.4)
- added REF**: MX_Cutout_1u, Keybage_MX_Cutout:MX_Cutout_1u, F.Cu at (57.1, 33.3)
- added REF**: MX_Cutout_1u, Keybage_MX_Cutout:MX_Cutout_1u, F.Cu at (57.1, 71.4)
- added REF**: MX_Cutout_1u, Keybage_MX_Cutout:MX_Cutout_1u, F.Cu at (57.1, -4.76)
- added REF**: MX_Cutout_1u, Keybage_MX_Cutout:MX_Cutout_1u, F.Cu at (57.1, 14.3)
- added REF**: MX_Cutout_1u, Keybage_MX_Cutout:MX_Cutout_1u, F.Cu at (38.1, 54.8)
- added REF**: MX_Cutout_1u, Keybage_MX_Cutout:MX_Cutout_1u, F.Cu at (38.1, 35.7)
- added REF**: MX_Cutout_1u, Keybage_MX_Cutout:MX_Cutout_1u, F.Cu at (38.1, 73.8)
- added REF**: MX_Cutout_1u, Keybage_MX_Cutout:MX_Cutout_1u, F.Cu at (38.1, -2.38)
- added REF**: MX_Cutout_1u, Keybage_MX_Cutout:MX_Cutout_1u, F.Cu at (19.1, 0.00)
- added REF**: MX_Cutout_1u, Keybage_MX_Cutout:MX_Cutout_1u, F.Cu at (19.1, 76.2)
- added REF**: MX_Cutout_1u, Keybage_MX_Cutout:MX_Cutout_1u, F.Cu at (19.1, 38.1)
- added REF**: MX_Cutout_1u, Keybage_MX_Cutout:MX_Cutout_1u, F.Cu at (19.1, 57.1)
- added REF**: MX_Cutout_1u, Keybage_MX_Cutout:MX_Cutout_1u, F.Cu at (19.1, 19.1)
- added REF**: MX_Cutout_1u, Keybage_MX_Cutout:MX_Cutout_1u, F.Cu at (0.00, 76.2)
- added REF**: MX_Cutout_1u, Keybage_MX_Cutout:MX_Cutout_1u, F.Cu at (0.00, 119.1)
- added REF**: MX_Cutout_1u, Keybage_MX_Cutout:MX_Cutout_1u, F.Cu at (0.00, 38.1)
- added REF**: MX_Cutout_1u, Keybage_MX_Cutout:MX_Cutout_1u, F.Cu at (0.00, 57.1)
- added REF**: MX_Cutout_1u, Keybage_MX_Cutout:MX_Cutout_1u, F.Cu at (0.00, 19.1)
- added REF**: MX_Cutout_1u, Keybage_MX_Cutout:MX_Cutout_1u, F.Cu at (0.00, 0.00)
- added REF**: MX_Cutout_1u, Keybage_MX_Cutout:MX_Cutout_1u, F.Cu at (38.1, 119.1)
- added REF**: MX_Cutout_1u, Keybage_MX_Cutout:MX_Cutout_1u, F.Cu at (19.1, 119.1)
- added REF**: MX_Cutout_1u, Keybage_MX_Cutout:MX_Cutout_1u, F.Cu at (19.1, 100.0)
- added REF**: MX_Cutout_1.25u, Keybage_MX_Cutout:MX_Cutout_1.25u, F.Cu at (76.2, 114.3)
- added REF**: MX_Cutout_1.25u, Keybage_MX_Cutout:MX_Cutout_1.25u, F.Cu at (95.2, 116.7)
Other:
- board outline added: 133.3 x 142.9 mm
