File: pcbfiles/_autosave-pcb.kicad_pcb (KiCad board)
At the start: 2 copper layers, 269.9 x 139.7 mm, 256 parts, among them J1 Conn_01x06, J2 Conn_01x06, J3 Conn_01x06, J4 Conn_01x06, J5 Conn_01x04_Female, J6 Conn_01x04_Female, Q1 AO3401A, Q2 AO3401A, SW1 SW_SPST, SW10 SW_SPST, SW11 SW_SPST, SW12 SW_SPST, SW13 SW_SPST, SW14 SW_SPST, SW15 SW_SPST, SW16 SW_SPST, SW17 SW_SPST, SW18 SW_SPST, SW19 SW_SPST, SW2 SW_SPST, SW20 SW_SPST, SW21 SW_SPST, SW22 SW_SPST, SW23 SW_SPST, SW24 SW_SPST, SW25 SW_SPST, SW26 SW_SPST, SW27 SW_SPST, SW28 SW_SPST, SW29 SW_SPST, SW3 SW_SPST, SW30 SW_SPST, SW31 SW_SPST, SW32 SW_SPST, SW33 SW_SPST, SW34 SW_SPST, SW35 SW_SPST, SW36 SW_SPST, SW37 SW_SPST, SW38 SW_SPST, SW39 SW_SPST, SW4 SW_SPST, SW40 SW_SPST, SW41 SW_SPST, SW42 SW_SPST, SW43 SW_SPST, SW44 SW_SPST, SW45 SW_SPST, SW46 SW_SPST, SW47 SW_SPST, SW48 SW_SPST, SW49 SW_SPST, SW5 SW_SPST, SW50 SW_SPST, SW51 SW_SPST, SW52 SW_SPST, SW53 SW_SPST, SW54 SW_SPST, SW55 SW_SPST, SW56 SW_SPST, SW57 SW_SPST, SW58 SW_SPST, SW59 SW_SPST, SW6 SW_SPST, SW60 SW_SPST, SW61 SW_SPST, SW62 SW_SPST, SW63 SW_SPST, SW64 SW_SPST, SW65 SW_SPST, SW66 SW_SPST, SW67 SW_SPST, SW68 SW_SPST, SW69 SW_SPST, SW7 SW_SPST, SW70 SW_SPST, SW71 SW_SPST, SW72 SW_SPST, SW73 SW_SPST, SW74 SW_SPST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

Commit message: quite a bit of routing
Routing:
- net DBA_P2: track 10.9 -> 43.9 mm
- net DBA_P5: track 44.7 -> 43.3 mm
- net DBA_P4: track 43.9 -> 43.2 mm
- net DBA_P1: track 44.8 -> 44.1 mm
Changed lines of the file:
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@@
   (segment (start -2.75 56) (end -2.75 54.9) (width 0.25) (layer "B.Cu") (net 200))
   (segment (start -3.85 54.9) (end -3.85 56) (width 0.25) (layer "B.Cu") (net 201))
-  (segment (start 37.1875 47.4) (end 35.3 47.4) (width 0.25) (layer "B.Cu") (net 213))
+  (segment (start 36.6875 47.4) (end 35.3 47.4) (width 0.25) (layer "B.Cu") (net 213))
   (segment (start 3.55 50.4) (end 32.8 50.4) (width 0.25) (layer "B.Cu") (net 213))
   (segment (start 33.3 49.4) (end 33.3 49.9) (width 0.25) (layer "B.Cu") (net 213))
-  (segment (start 37.1875 46.41875) (end 37.1875 47.4) (width 0.25) (layer "B.Cu") (net 213))
+  (segment (start 37.1875 46.41875) (end 37.1875 46.9) (width 0.25) (layer "B.Cu") (net 213))
   (segment (start 0.55 56) (end 0.55 53.4) (width 0.25) (layer "B.Cu") (net 213))
+  (arc (start 36.6875 47.4) (mid 37.041053 47.253553) (end 37.1875 46.9) (width 0.25) (layer "B.Cu") (net 213))
   (arc (start 0.55 53.4) (mid 1.42868 51.27868) (end 3.55 50.4) (width 0.25) (layer "B.Cu") (net 213))
   (arc (start 33.3 49.9) (mid 33.153553 50.253553) (end 32.8 50.4) (width 0.25) (layer "B.Cu") (net 213))
   (arc (start 35.3 47.4) (mid 33.885786 47.985786) (end 33.3 49.4) (width 0.25) (layer "B.Cu") (net 213))
-  (segment (start 38.1875 47.9) (end 38.1875 46.41875) (width 0.25) (layer "B.Cu") (net 214))
-  (segment (start 35.3 47.9) (end 38.1875 47.9) (width 0.25) (layer "B.Cu") (net 214))
+  (segment (start 38.1875 46.9) (end 38.1875 46.41875) (width 0.25) (layer "B.Cu") (net 214))
+  (segment (start 35.3 47.9) (end 37.1875 47.9) (width 0.25) (layer "B.Cu") (net 214))
   (segment (start 4.15 50.9) (end 32.8 50.9) (width 0.25) (layer "B.Cu") (net 214))
   (segment (start 33.8 49.9) (end 33.8 49.4) (width 0.25) (layer "B.Cu") (net 214))
   (segment (start 1.65 56) (end 1.65 53.4) (width 0.25) (layer "B.Cu") (net 214))
-  (segment (start 38.1875 46.41875) (end 38.1875 47.3125) (width 0.25) (layer "B.Cu") (net 214))
   (arc (start 33.8 49.4) (mid 34.23934 48.33934) (end 35.3 47.9) (width 0.25) (layer "B.Cu") (net 214))
+  (arc (start 37.1875 47.9) (mid 37.894607 47.607107) (end 38.1875 46.9) (width 0.25) (layer "B.Cu") (net 214))
   (arc (start 32.8 50.9) (mid 33.507107 50.607107) (end 33.8 49.9) (width 0.25) (layer "B.Cu") (net 214))
   (arc (start 1.65 53.4) (mid 2.382233 51.632233) (end 4.15 50.9) (width 0.25) (layer "B.Cu") (net 214))
   (segment (start 34.3 49.4) (end 34.3 49.9) (width 0.25) (layer "B.Cu") (net 215))
   (segment (start 32.8 51.4) (end 4.75 51.4) (width 0.25) (layer "B.Cu") (net 215))
-  (segment (start 39.1875 46.41875) (end 39.1875 48.4) (width 0.25) (layer "B.Cu") (net 215))
+  (segment (start 39.1875 46.41875) (end 39.1875 46.9) (width 0.25) (layer "B.Cu") (net 215))
   (segment (start 2.75 56) (end 2.75 53.4) (width 0.25) (layer "B.Cu") (net 215))
-  (segment (start 39.1875 48.4) (end 35.3 48.4) (width 0.25) (layer "B.Cu") (net 215))
+  (segment (start 37.6875 48.4) (end 35.3 48.4) (width 0.25) (layer "B.Cu") (net 215))
   (arc (start 4.75 51.4) (mid 3.335786 51.985786) (end 2.75 53.4) (width 0.25) (layer "B.Cu") (net 215))
   (arc (start 34.3 49.9) (mid 33.86066 50.96066) (end 32.8 51.4) (width 0.25) (layer "B.Cu") (net 215))
   (arc (start 35.3 48.4) (mid 34.592893 48.692893) (end 34.3 49.4) (width 0.25) (layer "B.Cu") (net 215))
-  (segment (start 39.1875 48.9) (end 35.3 48.9) (width 0.25) (layer "B.Cu") (net 216))
+  (arc (start 37.6875 48.4) (mid 38.74816 47.96066) (end 39.1875 46.9) (width 0.25) (layer "B.Cu") (net 215))
+  (segment (start 38.1875 48.9) (end 35.3 48.9) (width 0.25) (layer "B.Cu") (net 216))
   (segment (start 34.8 49.4) (end 34.8 49.89904) (width 0.25) (layer "B.Cu") (net 216))
-  (segment (start 40.1875 46.41875) (end 40.1875 47.9) (width 0.25) (layer "B.Cu") (net 216))
+  (segment (start 40.1875 46.41875) (end 40.1875 46.9) (width 0.25) (layer "B.Cu") (net 216))
   (segment (start 27.89952 51.89952) (end 27.9 51.89904) (width 0.25) (layer "B.Cu") (net 216))
   (segment (start 5.85 51.9) (end 25.2 51.9) (width 0.25) (layer "B.Cu") (net 216))
@@
   (segment (start 3.85 56) (end 3.85 53.9) (width 0.25) (layer "B.Cu") (net 216))
   (segment (start 27.9 51.89904) (end 25.60096 51.89904) (width 0.25) (layer "B.Cu") (net 216))
+  (arc (start 38.1875 48.9) (mid 39.601714 48.314214) (end 40.1875 46.9) (width 0.25) (layer "B.Cu") (net 216))
   (arc (start 34.8 49.89904) (mid 34.214214 51.313254) (end 32.8 51.89904) (width 0.25) (layer "B.Cu") (net 216))
   (arc (start 35.3 48.9) (mid 34.946447 49.046447) (end 34.8 49.4) (width 0.25) (layer "B.Cu") (net 216))
-  (arc (start 40.1875 47.9) (mid 39.894607 48.607107) (end 39.1875 48.9) (width 0.25) (layer "B.Cu") (net 216))
   (arc (start 3.85 53.9) (mid 4.435786 52.485786) (end 5.85 51.9) (width 0.25) (layer "B.Cu") (net 216))
-  (segment (start 41.1875 46.41875) (end 41.1875 51.4) (width 0.25) (layer "B.Cu") (net 217))
-  (segment (start 4.95 56) (end 4.95 53.9) (width 0.25) (layer "B.Cu") (net 217))
+  (segment (start 36.975 51.4) (end 36.975 50.9) (width 0.25) (layer "B.Cu") (net 217))
+  (segment (start 4.95 53.9) (end 4.95 56) (width 0.25) (layer "B.Cu") (net 217))
+  (segment (start 35.975 52.4) (end 6.45 52.4) (width 0.25) (layer "B.Cu") (net 217))
+  (segment (start 41.1875 46.41875) (end 41.1875 49.4) (width 0.25) (layer "B.Cu") (net 217))
+  (segment (start 41.1875 49.4) (end 38.475 49.4) (width 0.25) (layer "B.Cu") (net 217))
   (arc (start 6.45 52.4) (mid 5.38934 52.83934) (end 4.95 53.9) (width 0.25) (layer "B.Cu") (net 217))
-  (arc (start 40.1875 52.4) (mid 40.894607 52.107107) (end 41.1875 51.4) (width 0.25) (layer "B.Cu") (net 217))
-  (segment (start 7.05 52.9) (end 41.1875 52.9) (width 0.25) (layer "B.Cu") (net 218))
-  (segment (start 42.1875 51.9) (end 42.1875 46.41875) (width 0.25) (layer "B.Cu") (net 218))
+  (arc (start 36.975 51.4) (mid 36.682107 52.107107) (end 35.975 52.4) (width 0.25) (layer "B.Cu") (net 217))
+  (arc (start 38.475 49.4) (mid 37.41434 49.83934) (end 36.975 50.9) (width 0.25) (layer "B.Cu") (net 217))
+  (segment (start 42.1875 49.9) (end 38.5 49.9) (width 0.25) (layer "B.Cu") (net 218))
+  (segment (start 7.05 52.9) (end 36 52.9) (width 0.25) (layer "B.Cu") (net 218))
+  (segment (start 37.5 50.9) (end 37.5 51.4) (width 0.25) (layer "B.Cu") (net 218))
+  (segment (start 42.1875 46.41875) (end 42.1875 49.9) (width 0.25) (layer "B.Cu") (net 218))
   (segment (start 6.05 56) (end 6.05 53.9) (width 0.25) (layer "B.Cu") (net 218))
-  (arc (start 41.1875 52.9) (mid 41.894607 52.607107) (end 42.1875 51.9) (width 0.25) (layer "B.Cu") (net 218))
+  (arc (start 38.5 49.9) (mid 37.792893 50.192893) (end 37.5 50.9) (width 0.25) (layer "B.Cu") (net 218))
+  (arc (start 37.5 51.4) (mid 37.06066 52.46066) (end 36 52.9) (width 0.25) (layer "B.Cu") (net 218))
   (arc (start 7.05 52.9) (mid 6.342893 53.192893) (end 6.05 53.9) (width 0.25) (layer "B.Cu") (net 218))
   (zone (net 0) (net_name "") (layer "F.Cu") (hatch edge 0.508)
