File: pcbfiles/matrix-right.kicad_sch (KiCad schematic)
At the start: 72 parts, among them SW57 SW_SPST, SW58 SW_SPST, SW59 SW_SPST, SW60 SW_SPST, SW61 SW_SPST, SW62 SW_SPST, SW63 SW_SPST, SW64 SW_SPST, SW65 SW_SPST, SW67 SW_SPST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

Commit message: Making really good progress on the left half.
Parts:
- renumbered D58 to D59, D59 to D60, SW57 to SW59, SW58 to SW60, SW59 to SW61, SW60 to SW62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
