File: pcbfiles/pcb.kicad_sch (KiCad schematic)
At the start: 236 parts, among them J1 Conn_01x06, J2 Conn_01x06, J3 Conn_01x06, J4 Conn_01x06, J5 Conn_01x04_Female, J6 Conn_01x04_Female, Q1 AO3401A, Q2 AO3401A, SW1 SW_SPST, SW10 SW_SPST, SW11 SW_SPST, SW12 SW_SPST, SW13 SW_SPST, SW14 SW_SPST, SW15 SW_SPST, SW16 SW_SPST, SW17 SW_SPST, SW18 SW_SPST, SW19 SW_SPST, SW2 SW_SPST, SW20 SW_SPST, SW21 SW_SPST, SW22 SW_SPST, SW23 SW_SPST, SW24 SW_SPST, SW25 SW_SPST, SW26 SW_SPST, SW27 SW_SPST, SW28 SW_SPST, SW29 SW_SPST, SW3 SW_SPST, SW30 SW_SPST, SW31 SW_SPST, SW32 SW_SPST, SW33 SW_SPST, SW34 SW_SPST, SW35 SW_SPST, SW36 SW_SPST, SW37 SW_SPST, SW38 SW_SPST, SW39 SW_SPST, SW4 SW_SPST, SW40 SW_SPST, SW41 SW_SPST, SW42 SW_SPST, SW43 SW_SPST, SW44 SW_SPST, SW45 SW_SPST, SW46 SW_SPST, SW47 SW_SPST, SW48 SW_SPST, SW49 SW_SPST, SW5 SW_SPST, SW50 SW_SPST, SW51 SW_SPST, SW52 SW_SPST, SW53 SW_SPST, SW54 SW_SPST, SW55 SW_SPST, SW56 SW_SPST, SW57 SW_SPST, SW58 SW_SPST, SW59 SW_SPST, SW6 SW_SPST, SW60 SW_SPST, SW61 SW_SPST, SW62 SW_SPST, SW63 SW_SPST, SW64 SW_SPST, SW65 SW_SPST, SW66 SW_SPST, SW67 SW_SPST, SW68 SW_SPST, SW69 SW_SPST, SW7 SW_SPST, SW70 SW_SPST, SW71 SW_SPST, SW72 SW_SPST, SW73 SW_SPST, SW74 SW_SPST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

Commit message: switch placement right side preliminary
Parts:
- added D55: D_Small, Diode_SMD:D_SOD-123, symbol Device:D_Small
- added SW55: SW_SPST, MX_Only:MXOnly-1U-Hotswap, symbol Switch:SW_SPST
- SW74: renamed from SW73; footprint MX_Only:MXOnly-1U-Hotswap -> MX_Only:MXOnly-2.75U-Hotswap-ReversedStabilizers
- SW75: renamed from SW74; footprint MX_Only:MXOnly-1U-Hotswap -> MX_Only:MXOnly-1.25U-Hotswap
- SW76: renamed from SW75; footprint MX_Only:MXOnly-1U-Hotswap -> MX_Only:MXOnly-1.25U-Hotswap
- SW77: renamed from SW76; footprint MX_Only:MXOnly-1U-Hotswap -> MX_Only:MXOnly-1.25U-Hotswap
- renumbered D55 to D56, D56 to D57, D57 to D58, D58 to D59, D59 to D60, D60 to D61, D61 to D62, D62 to D63, D63 to D64, D64 to D65, D65 to D66, D66 to D67, D67 to D68, D68 to D69, D69 to D70, D70 to D71, D71 to D72, D72 to D73, D73 to D74, D74 to D75, D75 to D76, D76 to D77, D77 to D78, D78 to D79, D79 to D80, D80 to D81, D81 to D82, D82 to D83, D83 to D84, D84 to D85, D85 to D86, D86 to D87, D87 to D88, D88 to D89, D89 to D90, D90 to D91, D91 to D92, D92 to D93, D93 to D94, D94 to D95, SW55 to SW56, SW56 to SW57, SW57 to SW58, SW58 to SW59, SW59 to SW60, SW60 to SW61, SW61 to SW62, SW62 to SW63, SW63 to SW64, SW64 to SW65, SW65 to SW66, SW66 to SW67, SW67 to SW68, SW68 to SW69, SW69 to SW70, SW70 to SW71, SW71 to SW72, SW72 to SW73, SW77 to SW78, SW78 to SW79, SW79 to SW80, SW80 to SW81, SW81 to SW82, SW82 to SW83, SW83 to SW84, SW84 to SW85, SW85 to SW86, SW86 to SW87, SW87 to SW88, SW88 to SW89, SW89 to SW90, SW90 to SW91, SW91 to SW92, SW92 to SW93, SW93 to SW94, SW94 to SW95
Connections:
- net RH_ROW3: now also D55.1 (K)
- net at SW14.1 (A), SW28.1 (A), SW42.1 (A)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: now also SW55.1 (A)
- new net: D55.2 (A), SW55.2 (B)

Commit message: edgecuts and switches
Parts:
- SW72: footprint MX_Only:MXOnly-2U-Hotswap-ReversedStabilizers -> MX_Only:MXOnly-2U-Hotswap
- SW78, SW79, SW80: footprint MX_Only:MXOnly-1U-Hotswap -> MX_Only:MXOnly-1.25U-Hotswap
- SW81: footprint MX_Only:MXOnly-1U-Hotswap -> MX_Only:MXOnly-2.25U-Hotswap-ReversedStabilizers
Changed lines of the file:
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@@
     (property "Reference" "SW81" (id 0) (at 559.562 97.917 0))
     (property "Value" "SW_SPST" (id 1) (at 559.562 100.2284 0))
-    (property "Footprint" "MX_Only:MXOnly-1U-Hotswap" (id 2) (at 559.562 103.886 0)
+    (property "Footprint" "MX_Only:MXOnly-2.25U-Hotswap-ReversedStabilizers" (id 2) (at 559.562 103.886 0)
       (effects (font (size 1.27 1.27)) hide)
     )
@@
     (property "Reference" "SW72" (id 0) (at 577.342 80.645 0))
     (property "Value" "SW_SPST" (id 1) (at 577.342 82.9564 0))
-    (property "Footprint" "MX_Only:MXOnly-2U-Hotswap-ReversedStabilizers" (id 2) (at 577.342 86.614 0)
+    (property "Footprint" "MX_Only:MXOnly-2U-Hotswap" (id 2) (at 577.342 86.614 0)
       (effects (font (size 1.27 1.27)) hide)
     )
@@
     (property "Reference" "SW79" (id 0) (at 524.002 97.917 0))
     (property "Value" "SW_SPST" (id 1) (at 524.002 100.2284 0))
-    (property "Footprint" "MX_Only:MXOnly-1U-Hotswap" (id 2) (at 524.002 103.886 0)
+    (property "Footprint" "MX_Only:MXOnly-1.25U-Hotswap" (id 2) (at 524.002 103.886 0)
       (effects (font (size 1.27 1.27)) hide)
     )
@@
     (property "Reference" "SW80" (id 0) (at 541.782 97.917 0))
     (property "Value" "SW_SPST" (id 1) (at 541.782 100.2284 0))
-    (property "Footprint" "MX_Only:MXOnly-1U-Hotswap" (id 2) (at 541.782 103.886 0)
+    (property "Footprint" "MX_Only:MXOnly-1.25U-Hotswap" (id 2) (at 541.782 103.886 0)
       (effects (font (size 1.27 1.27)) hide)
     )
@@
     (property "Reference" "SW78" (id 0) (at 506.222 97.917 0))
     (property "Value" "SW_SPST" (id 1) (at 506.222 100.2284 0))
-    (property "Footprint" "MX_Only:MXOnly-1U-Hotswap" (id 2) (at 506.222 103.886 0)
+    (property "Footprint" "MX_Only:MXOnly-1.25U-Hotswap" (id 2) (at 506.222 103.886 0)
       (effects (font (size 1.27 1.27)) hide)
     )
@@
     )
     (path "/4173fd77-51b6-4d96-a24a-e3a75a365b7f"
-      (reference "SW72") (unit 1) (value "SW_SPST") (footprint "MX_Only:MXOnly-2U-Hotswap-ReversedStabilizers")
+      (reference "SW72") (unit 1) (value "SW_SPST") (footprint "MX_Only:MXOnly-2U-Hotswap")
     )
     (path "/497bc44f-43cd-4a3b-9323-f81df34db7dd"
@@
     )
     (path "/fa71d399-44a8-43ee-8505-9d9bfcc53b5f"
-      (reference "SW78") (unit 1) (value "SW_SPST") (footprint "MX_Only:MXOnly-1U-Hotswap")
+      (reference "SW78") (unit 1) (value "SW_SPST") (footprint "MX_Only:MXOnly-1.25U-Hotswap")
     )
     (path "/79f285c9-e8bd-48b4-8480-aeff2d68612f"
-      (reference "SW79") (unit 1) (value "SW_SPST") (footprint "MX_Only:MXOnly-1U-Hotswap")
+      (reference "SW79") (unit 1) (value "SW_SPST") (footprint "MX_Only:MXOnly-1.25U-Hotswap")
     )
     (path "/a74fc6b2-857d-4493-8915-1506601d4743"
-      (reference "SW80") (unit 1) (value "SW_SPST") (footprint "MX_Only:MXOnly-1U-Hotswap")
+      (reference "SW80") (unit 1) (value "SW_SPST") (footprint "MX_Only:MXOnly-1.25U-Hotswap")
     )
     (path "/125bb8dd-745e-4b63-82d5-102aaca46205"
-      (reference "SW81") (unit 1) (value "SW_SPST") (footprint "MX_Only:MXOnly-1U-Hotswap")
+      (reference "SW81") (unit 1) (value "SW_SPST") (footprint "MX_Only:MXOnly-2.25U-Hotswap-ReversedStabilizers")
     )
     (path "/5b145c59-359c-4ad1-9968-7874051fd0d2"

Commit message: progress on placement, some routing, encoders
Parts:
- removed H1, H2: MountingHole_Pad, symbol Mechanical:MountingHole_Pad
- SW74: footprint MX_Only:MXOnly-2.75U-Hotswap-ReversedStabilizers -> MX_Only:MXOnly-2.75U-Hotswap
- SW81: footprint MX_Only:MXOnly-2.25U-Hotswap-ReversedStabilizers -> MX_Only:MXOnly-2.25U-Hotswap
- renumbered C2 to C1, C1 to C2, D94 to D96, D95 to D97, F2 to F1, F1 to F2, R8 to R10, R9 to R11, R10 to R12, R11 to R13, R12 to R14, R13 to R15, R14 to R16, R15 to R17, R16 to R18, R6 to R5, R5 to R7, R7 to R9, SW93 to SW92, SW94 to SW93, SW92 to SW94, U4 to U3, U3 to U4
Connections:
- net RH_COL0 is gone; now on net ENC_P1_B: U6.4 (P1.13)
- net ENC_P1: now also SW90.S2; no longer SW90.S1
- net ENC_P2: now also SW90.S1; no longer SW90.S2
- net RH_COL1: now also SW23.1 (A), SW37.1 (A), SW50.1 (A), SW62.1 (A), SW71.1 (A), SW9.1 (A)
- net RH_COL2: now also SW10.1 (A), SW24.1 (A), SW38.1 (A), SW51.1 (A), SW63.1 (A)
- net RH_COL3: now also SW11.1 (A), SW25.1 (A), SW39.1 (A), SW52.1 (A), SW64.1 (A)
- net RH_COL4: now also SW12.1 (A), SW26.1 (A), SW40.1 (A), SW53.1 (A), SW65.1 (A)
- net RH_COL5: now also SW13.1 (A), SW27.1 (A), SW41.1 (A), SW54.1 (A), SW66.1 (A), SW72.1 (A)
- net RH_COL6: now also SW14.1 (A), SW28.1 (A), SW42.1 (A), SW55.1 (A), SW67.1 (A), SW73.1 (A)
- net VBAT_B: now also Q2.3 (D)
Other:
- moved on the sheet: BT1, BT2, C1, D97, F1, R18, R5, SW94, U3
