File: pcbfiles/pcb.kicad_sch (KiCad schematic)
At the start: 236 parts, among them J1 Conn_01x06, J2 Conn_01x06, J3 Conn_01x06, J4 Conn_01x06, J5 Conn_01x04_Female, J6 Conn_01x04_Female, Q1 AO3401A, Q2 AO3401A, SW1 SW_SPST, SW10 SW_SPST, SW11 SW_SPST, SW12 SW_SPST, SW13 SW_SPST, SW14 SW_SPST, SW15 SW_SPST, SW16 SW_SPST, SW17 SW_SPST, SW18 SW_SPST, SW19 SW_SPST, SW2 SW_SPST, SW20 SW_SPST, SW21 SW_SPST, SW22 SW_SPST, SW23 SW_SPST, SW24 SW_SPST, SW25 SW_SPST, SW26 SW_SPST, SW27 SW_SPST, SW28 SW_SPST, SW29 SW_SPST, SW3 SW_SPST, SW30 SW_SPST, SW31 SW_SPST, SW32 SW_SPST, SW33 SW_SPST, SW34 SW_SPST, SW35 SW_SPST, SW36 SW_SPST, SW37 SW_SPST, SW38 SW_SPST, SW39 SW_SPST, SW4 SW_SPST, SW40 SW_SPST, SW41 SW_SPST, SW42 SW_SPST, SW43 SW_SPST, SW44 SW_SPST, SW45 SW_SPST, SW46 SW_SPST, SW47 SW_SPST, SW48 SW_SPST, SW49 SW_SPST, SW5 SW_SPST, SW50 SW_SPST, SW51 SW_SPST, SW52 SW_SPST, SW53 SW_SPST, SW54 SW_SPST, SW55 SW_SPST, SW56 SW_SPST, SW57 SW_SPST, SW58 SW_SPST, SW59 SW_SPST, SW6 SW_SPST, SW60 SW_SPST, SW61 SW_SPST, SW62 SW_SPST, SW63 SW_SPST, SW64 SW_SPST, SW65 SW_SPST, SW66 SW_SPST, SW67 SW_SPST, SW68 SW_SPST, SW69 SW_SPST, SW7 SW_SPST, SW70 SW_SPST, SW71 SW_SPST, SW72 SW_SPST, SW73 SW_SPST, SW74 SW_SPST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

Commit message: Routing progress.
Connections:
- net LH_ROW0: now also U5.3 (P1.10)
- net LH_ROW1: now also U5.2 (P1.11)
- net LH_ROW2: now also U5.4 (P1.13)
Changed lines of the file:
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@@
+    )
+  )
+  (global_label "LH_ROW1" (shape input) (at 36.322 247.65 180) (fields_autoplaced)
+    (effects (font (size 1.27 1.27)) (justify right))
+    (property "Intersheet References" "${INTERSHEET_REFS}" (id 0) (at -90.678 124.46 0)
+      (effects (font (size 1.27 1.27)) hide)
     )
   )
@@
     )
   )
+  (global_label "LH_ROW0" (shape input) (at 36.322 250.19 180) (fields_autoplaced)
+    (effects (font (size 1.27 1.27)) (justify right))
+    (property "Intersheet References" "${INTERSHEET_REFS}" (id 0) (at -90.678 137.16 0)
+      (effects (font (size 1.27 1.27)) hide)
+    )
+  )
   (global_label "ENC_A_B" (shape input) (at 497.84 129.032 180) (fields_autoplaced)
     (effects (font (size 1.27 1.27)) (justify right))
@@
       (effects (font (size 1.27 1.27)) hide)
     )
+  )
+  (global_label "LH_ROW2" (shape input) (at 36.322 252.73 180) (fields_autoplaced)
+    (effects (font (size 1.27 1.27)) (justify right))
+    (property "Intersheet References" "${INTERSHEET_REFS}" (id 0) (at -90.678 119.38 0)
+      (effects (font (size 1.27 1.27)) hide)
+    )

Commit message: practically done with the left half
Connections:
- net LH_COL1: now also U5.30 (P1.02)
- net LH_COL2: now also U5.29 (P1.01)
- net LH_COL3: now also U5.28 (P1.03)
- net LH_COL4: now also U5.27 (P1.00)
- net LH_COL5: now also U5.26 (P0.22)
Changed lines of the file:
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@@
+    )
+  )
+  (global_label "LH_COL1" (shape input) (at 71.882 262.89 0) (fields_autoplaced)
+    (effects (font (size 1.27 1.27)) (justify left))
+    (property "Intersheet References" "${INTERSHEET_REFS}" (id 0) (at 169.672 110.49 0)
+      (effects (font (size 1.27 1.27)) hide)
     )
   )
@@
     )
   )
+  (global_label "LH_COL5" (shape input) (at 71.882 273.05 0) (fields_autoplaced)
+    (effects (font (size 1.27 1.27)) (justify left))
+    (property "Intersheet References" "${INTERSHEET_REFS}" (id 0) (at 169.672 49.53 0)
+      (effects (font (size 1.27 1.27)) hide)
+    )
+  )
   (global_label "LH_ROW0" (shape input) (at 36.322 250.19 180) (fields_autoplaced)
     (effects (font (size 1.27 1.27)) (justify right))
@@
     (effects (font (size 1.27 1.27)) (justify left))
     (property "Intersheet References" "${INTERSHEET_REFS}" (id 0) (at 30.988 160.274 0)
+      (effects (font (size 1.27 1.27)) hide)
+    )
+  )
+  (global_label "LH_COL3" (shape input) (at 71.882 267.97 0) (fields_autoplaced)
+    (effects (font (size 1.27 1.27)) (justify left))
+    (property "Intersheet References" "${INTERSHEET_REFS}" (id 0) (at 169.672 80.01 0)
       (effects (font (size 1.27 1.27)) hide)
     )
@@
     )
   )
+  (global_label "LH_COL4" (shape input) (at 71.882 270.51 0) (fields_autoplaced)
+    (effects (font (size 1.27 1.27)) (justify left))
+    (property "Intersheet References" "${INTERSHEET_REFS}" (id 0) (at 169.672 64.77 0)
+      (effects (font (size 1.27 1.27)) hide)
+    )
+  )
   (global_label "RH_ROW3" (shape input) (at 510.032 288.29 270) (fields_autoplaced)
     (effects (font (size 1.27 1.27)) (justify right))
@@
       (effects (font (size 1.27 1.27)) hide)
     )
+  )
+  (global_label "LH_COL2" (shape input) (at 71.882 265.43 0) (fields_autoplaced)
+    (effects (font (size 1.27 1.27)) (justify left))
+    (property "Intersheet References" "${INTERSHEET_REFS}" (id 0) (at 169.672 95.25 0)
+      (effects (font (size 1.27 1.27)) hide)
+    )

Commit message: Routing.
Connections:
- net ENC_A: now also U5.16 (P1.09)
- net ENC_B: now also U5.17 (P0.12)
- net ENC_P1: now also U5.15 (P0.07)
- net LH_COL0: now also U5.33 (P1.04)
- net LH_ROW4: now also U5.35 (P0.09)
- net LH_ROW5: now also U5.36 (P0.10)
Changed lines of the file:
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@@
+    )
+  )
+  (global_label "ENC_B" (shape input) (at 49.022 288.29 270) (fields_autoplaced)
+    (effects (font (size 1.27 1.27)) (justify right))
+    (property "Intersheet References" "${INTERSHEET_REFS}" (id 0) (at 49.1014 296.6013 90)
+      (effects (font (size 1.27 1.27)) (justify right) hide)
     )
   )
@@
     )
   )
+  (global_label "LH_ROW5" (shape input) (at 71.882 247.65 0) (fields_autoplaced)
+    (effects (font (size 1.27 1.27)) (justify left))
+    (property "Intersheet References" "${INTERSHEET_REFS}" (id 0) (at 198.882 411.48 0)
+      (effects (font (size 1.27 1.27)) hide)
+    )
+  )
+  (global_label "LH_COL0" (shape input) (at 71.882 255.27 0) (fields_autoplaced)
+    (effects (font (size 1.27 1.27)) (justify left))
+    (property "Intersheet References" "${INTERSHEET_REFS}" (id 0) (at 82.3705 255.1906 0)
+      (effects (font (size 1.27 1.27)) (justify left) hide)
+    )
+  )
   (global_label "DBA_P3" (shape input) (at 36.322 265.43 180) (fields_autoplaced)
     (effects (font (size 1.27 1.27)) (justify right))
@@
     )
   )
+  (global_label "ENC_A" (shape input) (at 46.482 288.29 270) (fields_autoplaced)
+    (effects (font (size 1.27 1.27)) (justify right))
+    (property "Intersheet References" "${INTERSHEET_REFS}" (id 0) (at 46.5614 296.4199 90)
+      (effects (font (size 1.27 1.27)) (justify right) hide)
+    )
+  )
   (global_label "VBUS_B" (shape input) (at 631.952 158.75 180) (fields_autoplaced)
     (effects (font (size 1.27 1.27)) (justify right))
     (property "Intersheet References" "${INTERSHEET_REFS}" (id 0) (at 60.452 128.27 0)
+      (effects (font (size 1.27 1.27)) hide)
+    )
+  )
+  (global_label "LH_ROW4" (shape input) (at 71.882 250.19 0) (fields_autoplaced)
+    (effects (font (size 1.27 1.27)) (justify left))
+    (property "Intersheet References" "${INTERSHEET_REFS}" (id 0) (at 198.882 403.86 0)
       (effects (font (size 1.27 1.27)) hide)
     )
@@
       (effects (font (size 1.27 1.27)) hide)
     )
+  )
+  (global_label "LH_COL6" (shape input) (at 43.942 288.29 270) (fields_autoplaced)
+    (effects (font (size 1.27 1.27)) (justify right))
+    (property "Intersheet References" "${INTERSHEET_REFS}" (id 0) (at 285.242 386.08 0)
+      (effects (font (size 1.27 1.27)) hide)
+    )

Commit message: Routing.
Connections:
- net ENC_A: now also U5.17 (P0.12); no longer U5.16 (P1.09)
- net ENC_B: now also U5.18 (P0.23); no longer U5.17 (P0.12)
- net ENC_P1: now also U5.16 (P1.09); no longer U5.15 (P0.07)
Changed lines of the file:
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@@
     )
   )
-  (global_label "ENC_B" (shape input) (at 49.022 288.29 270) (fields_autoplaced)
-    (effects (font (size 1.27 1.27)) (justify right))
-    (property "Intersheet References" "${INTERSHEET_REFS}" (id 0) (at 49.1014 296.6013 90)
+  (global_label "ENC_B" (shape input) (at 51.562 288.29 270) (fields_autoplaced)
+    (effects (font (size 1.27 1.27)) (justify right))
+    (property "Intersheet References" "${INTERSHEET_REFS}" (id 0) (at 51.6414 296.6013 90)
       (effects (font (size 1.27 1.27)) (justify right) hide)
     )
@@
     )
   )
-  (global_label "ENC_A" (shape input) (at 46.482 288.29 270) (fields_autoplaced)
-    (effects (font (size 1.27 1.27)) (justify right))
-    (property "Intersheet References" "${INTERSHEET_REFS}" (id 0) (at 46.5614 296.4199 90)
+  (global_label "ENC_A" (shape input) (at 49.022 288.29 270) (fields_autoplaced)
+    (effects (font (size 1.27 1.27)) (justify right))
+    (property "Intersheet References" "${INTERSHEET_REFS}" (id 0) (at 49.1014 296.4199 90)
       (effects (font (size 1.27 1.27)) (justify right) hide)
     )
@@
     )
   )
-  (global_label "LH_COL6" (shape input) (at 43.942 288.29 270) (fields_autoplaced)
-    (effects (font (size 1.27 1.27)) (justify right))
-    (property "Intersheet References" "${INTERSHEET_REFS}" (id 0) (at 285.242 386.08 0)
-      (effects (font (size 1.27 1.27)) hide)
-    )
+  (global_label "LH_COL6" (shape input) (at 46.482 288.29 270) (fields_autoplaced)
+    (effects (font (size 1.27 1.27)) (justify right))
+    (property "Intersheet References" "${INTERSHEET_REFS}" (id 0) (at 287.782 386.08 0)
+      (effects (font (size 1.27 1.27)) hide)
+    )

Commit message: Routing.
Connections:
- net DBB_P1: now reaches J2.1 (Pin_1), J4.6 (Pin_6)
- net DBB_P2: now reaches J2.2 (Pin_2), J4.5 (Pin_5)
- net DBB_P3: now reaches J2.3 (Pin_3), J4.4 (Pin_4)
- net DBB_P4: now reaches J2.4 (Pin_4), J4.3 (Pin_3)
- net DBB_P5: now reaches J2.5 (Pin_5), J4.2 (Pin_2)
- net DBB_P6: now reaches J2.6 (Pin_6), J4.1 (Pin_1)
Changed lines of the file:
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@@
+    )
+  )
+  (global_label "DBB_P3" (shape input) (at 636.524 100.838 180) (fields_autoplaced)
+    (effects (font (size 1.27 1.27)) (justify right))
+    (property "Intersheet References" "${INTERSHEET_REFS}" (id 0) (at 626.9427 100.7586 0)
+      (effects (font (size 1.27 1.27)) (justify right) hide)
     )
   )
@@
     )
   )
+  (global_label "DBB_P6" (shape input) (at 644.144 108.458 180) (fields_autoplaced)
+    (effects (font (size 1.27 1.27)) (justify right))
+    (property "Intersheet References" "${INTERSHEET_REFS}" (id 0) (at 634.5627 108.3786 0)
+      (effects (font (size 1.27 1.27)) (justify right) hide)
+    )
+  )
   (global_label "ENC_B" (shape input) (at 51.562 288.29 270) (fields_autoplaced)
     (effects (font (size 1.27 1.27)) (justify right))
@@
     )
   )
+  (global_label "DBB_P4" (shape input) (at 639.064 103.378 180) (fields_autoplaced)
+    (effects (font (size 1.27 1.27)) (justify right))
+    (property "Intersheet References" "${INTERSHEET_REFS}" (id 0) (at 629.4827 103.2986 0)
+      (effects (font (size 1.27 1.27)) (justify right) hide)
+    )
+  )
   (global_label "RAW" (shape input) (at 111.252 153.67 180) (fields_autoplaced)
     (effects (font (size 1.27 1.27)) (justify right))
@@
     )
   )
+  (global_label "DBB_P5" (shape input) (at 641.604 105.918 180) (fields_autoplaced)
+    (effects (font (size 1.27 1.27)) (justify right))
+    (property "Intersheet References" "${INTERSHEET_REFS}" (id 0) (at 632.0227 105.8386 0)
+      (effects (font (size 1.27 1.27)) (justify right) hide)
+    )
+  )
   (global_label "RH_COL4" (shape input) (at 554.482 25.654 90) (fields_autoplaced)
     (effects (font (size 1.27 1.27)) (justify left))
@@
     )
   )
+  (global_label "DBB_P1" (shape input) (at 631.444 95.758 180) (fields_autoplaced)
+    (effects (font (size 1.27 1.27)) (justify right))
+    (property "Intersheet References" "${INTERSHEET_REFS}" (id 0) (at 621.8627 95.6786 0)
+      (effects (font (size 1.27 1.27)) (justify right) hide)
+    )
+  )
   (global_label "SWD_B" (shape input) (at 555.752 266.7 180) (fields_autoplaced)
     (effects (font (size 1.27 1.27)) (justify right))
@@
     )
   )
+  (global_label "DBB_P2" (shape input) (at 633.984 98.298 180) (fields_autoplaced)
+    (effects (font (size 1.27 1.27)) (justify right))
+    (property "Intersheet References" "${INTERSHEET_REFS}" (id 0) (at 624.4027 98.2186 0)
+      (effects (font (size 1.27 1.27)) (justify right) hide)
+    )
+  )

Commit message: Routing.
Connections:
- net ENC_P1_B: no longer U6.4 (P1.13)
- net RH_COL1: no longer U6.18 (P0.23)
- net RH_COL2: no longer U6.17 (P0.12)
- net RH_COL3: no longer U6.16 (P1.09), U6.7 (P0.02)
- net RH_COL4: no longer U6.15 (P0.07)
- net RH_COL5: no longer U6.35 (P0.09)
- net RH_ROW0: no longer U6.33 (P1.04)
- net RH_ROW1: no longer U6.34 (P1.06)
- net RH_ROW2: no longer U6.30 (P1.02)
- net RH_ROW3: no longer U6.20 (P0.19)
- net RH_ROW4: no longer U6.13 (P0.05)
- net RH_ROW5: no longer U6.6 (P0.03)
Changed lines of the file:
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@@
-    )
-  )
-  (global_label "RH_ROW0" (shape input) (at 525.272 255.27 0) (fields_autoplaced)
-    (effects (font (size 1.27 1.27)) (justify left))
-    (property "Intersheet References" "${INTERSHEET_REFS}" (id 0) (at 60.452 128.27 0)
-      (effects (font (size 1.27 1.27)) hide)
     )
   )
@@
     )
   )
-  (global_label "RH_COL3" (shape input) (at 499.872 288.29 270) (fields_autoplaced)
-    (effects (font (size 1.27 1.27)) (justify right))
-    (property "Intersheet References" "${INTERSHEET_REFS}" (id 0) (at 60.452 128.27 0)
-      (effects (font (size 1.27 1.27)) hide)
-    )
-  )
   (global_label "D-" (shape input) (at 64.262 288.29 270) (fields_autoplaced)
     (effects (font (size 1.27 1.27)) (justify right))
@@
     )
   )
-  (global_label "RH_COL4" (shape input) (at 497.332 288.29 270) (fields_autoplaced)
-    (effects (font (size 1.27 1.27)) (justify right))
-    (property "Intersheet References" "${INTERSHEET_REFS}" (id 0) (at 60.452 128.27 0)
-      (effects (font (size 1.27 1.27)) hide)
-    )
-  )
   (global_label "DBA_COL2" (shape input) (at 105.41 103.632 90) (fields_autoplaced)
     (effects (font (size 1.27 1.27)) (justify left))
@@
     (effects (font (size 1.27 1.27)) (justify left))
     (property "Intersheet References" "${INTERSHEET_REFS}" (id 0) (at 169.672 110.49 0)
-      (effects (font (size 1.27 1.27)) hide)
-    )
-  )
-  (global_label "RH_ROW2" (shape input) (at 525.272 262.89 0) (fields_autoplaced)
-    (effects (font (size 1.27 1.27)) (justify left))
-    (property "Intersheet References" "${INTERSHEET_REFS}" (id 0) (at 60.452 128.27 0)
       (effects (font (size 1.27 1.27)) hide)
     )
@@
     )
   )
-  (global_label "RH_COL5" (shape input) (at 525.272 250.19 0) (fields_autoplaced)
-    (effects (font (size 1.27 1.27)) (justify left))
-    (property "Intersheet References" "${INTERSHEET_REFS}" (id 0) (at 60.452 128.27 0)
-      (effects (font (size 1.27 1.27)) hide)
-    )
-  )
   (global_label "ENC_A" (shape input) (at 66.802 129.032 180) (fields_autoplaced)
     (effects (font (size 1.27 1.27)) (justify right))
@@
     )
   )
-  (global_label "RH_COL0" (shape input) (at 489.712 252.73 180) (fields_autoplaced)
-    (effects (font (size 1.27 1.27)) (justify right))
-    (property "Intersheet References" "${INTERSHEET_REFS}" (id 0) (at 60.452 128.27 0)
-      (effects (font (size 1.27 1.27)) hide)
-    )
-  )
-  (global_label "RH_ROW5" (shape input) (at 489.712 257.81 180) (fields_autoplaced)
-    (effects (font (size 1.27 1.27)) (justify right))
-    (property "Intersheet References" "${INTERSHEET_REFS}" (id 0) (at 60.452 128.27 0)
-      (effects (font (size 1.27 1.27)) hide)
-    )
-  )
   (global_label "DBA_P5" (shape input) (at 164.592 105.918 180) (fields_autoplaced)
     (effects (font (size 1.27 1.27)) (justify right))
@@
     (effects (font (size 1.27 1.27)) (justify right))
     (property "Intersheet References" "${INTERSHEET_REFS}" (id 0) (at 60.96 126.492 0)
-      (effects (font (size 1.27 1.27)) hide)
-    )
-  )
-  (global_label "RH_COL3" (shape input) (at 489.712 260.35 180) (fields_autoplaced)
-    (effects (font (size 1.27 1.27)) (justify right))
-    (property "Intersheet References" "${INTERSHEET_REFS}" (id 0) (at 60.452 128.27 0)
       (effects (font (size 1.27 1.27)) hide)
     )
@@
     )
   )
-  (global_label "RH_ROW3" (shape input) (at 510.032 288.29 270) (fields_autoplaced)
-    (effects (font (size 1.27 1.27)) (justify right))
-    (property "Intersheet References" "${INTERSHEET_REFS}" (id 0) (at 60.452 128.27 0)
-      (effects (font (size 1.27 1.27)) hide)
-    )
-  )
   (global_label "B_D-" (shape input) (at 531.622 156.21 0) (fields_autoplaced)
     (effects (font (size 1.27 1.27)) (justify left))
@@
     )
   )
-  (global_label "RH_COL1" (shape input) (at 504.952 288.29 270) (fields_autoplaced)
-    (effects (font (size 1.27 1.27)) (justify right))
-    (property "Intersheet References" "${INTERSHEET_REFS}" (id 0) (at 60.452 128.27 0)
-      (effects (font (size 1.27 1.27)) hide)
-    )
-  )
   (global_label "VBUS_B" (shape input) (at 555.752 259.08 180) (fields_autoplaced)
     (effects (font (size 1.27 1.27)) (justify right))
@@
     (effects (font (size 1.27 1.27)) (justify left))
     (property "Intersheet References" "${INTERSHEET_REFS}" (id 0) (at 60.96 126.492 0)
-      (effects (font (size 1.27 1.27)) hide)
-    )
-  )
-  (global_label "RH_COL2" (shape input) (at 502.412 288.29 270) (fields_autoplaced)
-    (effects (font (size 1.27 1.27)) (justify right))
-    (property "Intersheet References" "${INTERSHEET_REFS}" (id 0) (at 60.452 128.27 0)
       (effects (font (size 1.27 1.27)) hide)
     )
@@
     )
   )
-  (global_label "RH_ROW4" (shape input) (at 489.712 275.59 180) (fields_autoplaced)
-    (effects (font (size 1.27 1.27)) (justify right))
-    (property "Intersheet References" "${INTERSHEET_REFS}" (id 0) (at 60.452 128.27 0)
-      (effects (font (size 1.27 1.27)) hide)
-    )
-  )
   (global_label "BVOLT" (shape input) (at 36.322 273.05 180) (fields_autoplaced)
     (effects (font (size 1.27 1.27)) (justify right))
@@
       (effects (font (size 1.27 1.27)) hide)
     )
-  )
-  (global_label "RH_ROW1" (shape input) (at 525.272 252.73 0) (fields_autoplaced)
-    (effects (font (size 1.27 1.27)) (justify left))
-    (property "Intersheet References" "${INTERSHEET_REFS}" (id 0) (at 60.452 128.27 0)
-      (effects (font (size 1.27 1.27)) hide)
-    )

Commit message: Significant work on Routing.
right side!
Connections:
- net DBA_COL1: no longer D82.1 (K), D83.1 (K), D84.1 (K), D85.1 (K)
- net ENC_A_B: no longer U6.2 (P1.11)
- net ENC_B_B: no longer U6.3 (P1.10)
- net RH_COL1: now also U6.11 (P0.31)
- net RH_COL4: now also U6.26 (P0.22)
- net RH_COL5: now also U6.28 (P1.03)
- net RH_COL6: no longer U6.36 (P0.10)
- net RH_ROW4: now also U6.29 (P1.01)
- new net DBA_ROW1: D82.1 (K), D83.1 (K), D84.1 (K), D85.1 (K)
Changed lines of the file:
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@@
+    )
+  )
+  (global_label "RH_ROW4" (shape input) (at 525.272 265.43 0) (fields_autoplaced)
+    (effects (font (size 1.27 1.27)) (justify left))
+    (property "Intersheet References" "${INTERSHEET_REFS}" (id 0) (at 536.4257 265.3506 0)
+      (effects (font (size 1.27 1.27)) (justify left) hide)
     )
   )
@@
     )
   )
+  (global_label "RH_COL5" (shape input) (at 525.272 267.97 0) (fields_autoplaced)
+    (effects (font (size 1.27 1.27)) (justify left))
+    (property "Intersheet References" "${INTERSHEET_REFS}" (id 0) (at 536.0024 267.8906 0)
+      (effects (font (size 1.27 1.27)) (justify left) hide)
+    )
+  )
   (global_label "ENC_B" (shape input) (at 51.562 288.29 270) (fields_autoplaced)
     (effects (font (size 1.27 1.27)) (justify right))
@@
     )
   )
-  (global_label "ENC_B_B" (shape input) (at 489.712 250.19 180) (fields_autoplaced)
-    (effects (font (size 1.27 1.27)) (justify right))
-    (property "Intersheet References" "${INTERSHEET_REFS}" (id 0) (at 479.163 250.1106 0)
-      (effects (font (size 1.27 1.27)) (justify right) hide)
-    )
-  )
   (global_label "RH_COL3" (shape input) (at 536.702 25.654 90) (fields_autoplaced)
     (effects (font (size 1.27 1.27)) (justify left))
@@
     )
   )
+  (global_label "RH_COL4" (shape input) (at 525.272 273.05 0) (fields_autoplaced)
+    (effects (font (size 1.27 1.27)) (justify left))
+    (property "Intersheet References" "${INTERSHEET_REFS}" (id 0) (at 609.092 -336.55 0)
+      (effects (font (size 1.27 1.27)) hide)
+    )
+  )
   (global_label "RAW" (shape input) (at 49.022 180.34 0) (fields_autoplaced)
     (effects (font (size 1.27 1.27)) (justify left))
@@
     (effects (font (size 1.27 1.27)) (justify right))
     (property "Intersheet References" "${INTERSHEET_REFS}" (id 0) (at 13.462 128.27 0)
-      (effects (font (size 1.27 1.27)) hide)
-    )
-  )
-  (global_label "RH_COL6" (shape input) (at 525.272 247.65 0) (fields_autoplaced)
-    (effects (font (size 1.27 1.27)) (justify left))
-    (property "Intersheet References" "${INTERSHEET_REFS}" (id 0) (at 60.452 128.27 0)
       (effects (font (size 1.27 1.27)) hide)
     )
@@
     )
   )
-  (global_label "DBA_COL1" (shape input) (at 66.802 118.872 180) (fields_autoplaced)
-    (effects (font (size 1.27 1.27)) (justify right))
-    (property "Intersheet References" "${INTERSHEET_REFS}" (id 0) (at 55.0435 118.7926 0)
+  (global_label "DBA_ROW1" (shape input) (at 66.802 118.872 180) (fields_autoplaced)
+    (effects (font (size 1.27 1.27)) (justify right))
+    (property "Intersheet References" "${INTERSHEET_REFS}" (id 0) (at 54.6202 118.7926 0)
       (effects (font (size 1.27 1.27)) (justify right) hide)
     )
@@
     )
   )
-  (global_label "ENC_A_B" (shape input) (at 489.712 247.65 180) (fields_autoplaced)
-    (effects (font (size 1.27 1.27)) (justify right))
-    (property "Intersheet References" "${INTERSHEET_REFS}" (id 0) (at 479.3445 247.5706 0)
-      (effects (font (size 1.27 1.27)) (justify right) hide)
-    )
-  )
   (global_label "BVOLT_B" (shape input) (at 489.712 273.05 180) (fields_autoplaced)
     (effects (font (size 1.27 1.27)) (justify right))
@@
       (effects (font (size 1.27 1.27)) hide)
     )
+  )
+  (global_label "RH_COL1" (shape input) (at 489.712 270.51 180) (fields_autoplaced)
+    (effects (font (size 1.27 1.27)) (justify right))
+    (property "Intersheet References" "${INTERSHEET_REFS}" (id 0) (at 405.892 826.77 0)
+      (effects (font (size 1.27 1.27)) hide)
+    )

Commit message: Routing
Connections:
- net RH_COL4: now also U6.30 (P1.02)
- net RH_COL6: now also U6.36 (P0.10)
- net RH_ROW1: now also U6.33 (P1.04)
- net RH_ROW2: now also U6.34 (P1.06)
- net RH_ROW3: now also U6.35 (P0.09)
Changed lines of the file:
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@@
+    )
+  )
+  (global_label "RH_ROW2" (shape input) (at 525.272 252.73 0) (fields_autoplaced)
+    (effects (font (size 1.27 1.27)) (justify left))
+    (property "Intersheet References" "${INTERSHEET_REFS}" (id 0) (at -130.048 133.35 0)
+      (effects (font (size 1.27 1.27)) hide)
     )
   )
@@
     )
   )
+  (global_label "RH_ROW1" (shape input) (at 525.272 255.27 0) (fields_autoplaced)
+    (effects (font (size 1.27 1.27)) (justify left))
+    (property "Intersheet References" "${INTERSHEET_REFS}" (id 0) (at 536.4257 255.1906 0)
+      (effects (font (size 1.27 1.27)) (justify left) hide)
+    )
+  )
   (global_label "RAW_B" (shape input) (at 568.96 151.892 180) (fields_autoplaced)
     (effects (font (size 1.27 1.27)) (justify right))
@@
     )
   )
+  (global_label "RH_ROW3" (shape input) (at 525.272 250.19 0) (fields_autoplaced)
+    (effects (font (size 1.27 1.27)) (justify left))
+    (property "Intersheet References" "${INTERSHEET_REFS}" (id 0) (at -130.048 120.65 0)
+      (effects (font (size 1.27 1.27)) hide)
+    )
+  )
   (global_label "VBUS_B" (shape input) (at 574.548 163.322 90) (fields_autoplaced)
     (effects (font (size 1.27 1.27)) (justify left))
@@
     )
   )
+  (global_label "RH_COL4" (shape input) (at 525.272 262.89 0) (fields_autoplaced)
+    (effects (font (size 1.27 1.27)) (justify left))
+    (property "Intersheet References" "${INTERSHEET_REFS}" (id 0) (at 609.092 -346.71 0)
+      (effects (font (size 1.27 1.27)) hide)
+    )
+  )
   (global_label "VBAT" (shape input) (at 132.842 168.91 0) (fields_autoplaced)
     (effects (font (size 1.27 1.27)) (justify left))
@@
     )
   )
+  (global_label "RH_COL6" (shape input) (at 525.272 247.65 0) (fields_autoplaced)
+    (effects (font (size 1.27 1.27)) (justify left))
+    (property "Intersheet References" "${INTERSHEET_REFS}" (id 0) (at 609.092 -397.51 0)
+      (effects (font (size 1.27 1.27)) hide)
+    )
+  )
